File: _saved_FireMC-3.14_MTR.sch (KiCad schematic (older format))
At the start: 24 parts

Commit message: math check
Parts:
- removed J? (x4): Header_1X3, symbol Header_1X3
Changed lines of the file:
@@
 	1    0    0    -1
 $EndComp
-$Comp
-L Header_1X3 J?
-U 1 1 57D1A629
-P 3800 7500
-F 0 "J?" H 3800 7750 60  0000 C CNN
-F 1 "Header_1X3" H 3800 7250 60  0000 C CNN
-F 2 "" H 3800 7450 60  0000 C CNN
-F 3 "" H 3800 7450 60  0000 C CNN
-	1    3800 7500
-	-1   0    0    -1
-$EndComp
-$Comp
-L Header_1X3 J?
-U 1 1 57D1A749
-P 2800 7500
-F 0 "J?" H 2800 7750 60  0000 C CNN
-F 1 "Header_1X3" H 2800 7250 60  0000 C CNN
-F 2 "" H 2800 7450 60  0000 C CNN
-F 3 "" H 2800 7450 60  0000 C CNN
-	1    2800 7500
-	-1   0    0    -1
-$EndComp
-$Comp
-L Header_1X3 J?
-U 1 1 57D1A7FF
-P 1800 7500
-F 0 "J?" H 1800 7750 60  0000 C CNN
-F 1 "Header_1X3" H 1800 7250 60  0000 C CNN
-F 2 "" H 1800 7450 60  0000 C CNN
-F 3 "" H 1800 7450 60  0000 C CNN
-	1    1800 7500
-	-1   0    0    -1
-$EndComp
-$Comp
-L Header_1X3 J?
-U 1 1 57D1A87E
-P 800 7500
-F 0 "J?" H 800 7750 60  0000 C CNN
-F 1 "Header_1X3" H 800 7250 60  0000 C CNN
-F 2 "" H 800 7450 60  0000 C CNN
-F 3 "" H 800 7450 60  0000 C CNN
-	1    800  7500
-	-1   0    0    -1
-$EndComp
-$Comp
-L GND #PWR?
-U 1 1 57D1AB18
-P 1200 7700
-F 0 "#PWR?" H 1200 7450 50  0001 C CNN
-F 1 "GND" H 1200 7550 50  0000 C CNN
-F 2 "" H 1200 7700 50  0000 C CNN
-F 3 "" H 1200 7700 50  0000 C CNN
-	1    1200 7700
-	1    0    0    -1
-$EndComp
-$Comp
-L GND #PWR?
-U 1 1 57D1AB6B
-P 2200 7700
-F 0 "#PWR?" H 2200 7450 50  0001 C CNN
-F 1 "GND" H 2200 7550 50  0000 C CNN
-F 2 "" H 2200 7700 50  0000 C CNN
-F 3 "" H 2200 7700 50  0000 C CNN
-	1    2200 7700
-	1    0    0    -1
-$EndComp
-$Comp
-L GND #PWR?
-U 1 1 57D1ABBE
-P 3200 7700
-F 0 "#PWR?" H 3200 7450 50  0001 C CNN
-F 1 "GND" H 3200 7550 50  0000 C CNN
-F 2 "" H 3200 7700 50  0000 C CNN
-F 3 "" H 3200 7700 50  0000 C CNN
-	1    3200 7700
-	1    0    0    -1
-$EndComp
-$Comp
-L GND #PWR?
-U 1 1 57D1AC11
-P 4200 7700
-F 0 "#PWR?" H 4200 7450 50  0001 C CNN
-F 1 "GND" H 4200 7550 50  0000 C CNN
-F 2 "" H 4200 7700 50  0000 C CNN
-F 3 "" H 4200 7700 50  0000 C CNN
-	1    4200 7700
-	1    0    0    -1
-$EndComp
-$Comp
-L VCC #PWR?
-U 1 1 57D1AC64
-P 1200 7300
-F 0 "#PWR?" H 1200 7150 50  0001 C CNN
-F 1 "VCC" H 1200 7450 50  0000 C CNN
-F 2 "" H 1200 7300 50  0000 C CNN
-F 3 "" H 1200 7300 50  0000 C CNN
-	1    1200 7300
-	1    0    0    -1
-$EndComp
-$Comp
-L VCC #PWR?
-U 1 1 57D1ACB7
-P 2200 7300
-F 0 "#PWR?" H 2200 7150 50  0001 C CNN
-F 1 "VCC" H 2200 7450 50  0000 C CNN
-F 2 "" H 2200 7300 50  0000 C CNN
-F 3 "" H 2200 7300 50  0000 C CNN
-	1    2200 7300
-	1    0    0    -1
-$EndComp
-$Comp
-L VCC #PWR?
-U 1 1 57D1AD0A
-P 3200 7300
-F 0 "#PWR?" H 3200 7150 50  0001 C CNN
-F 1 "VCC" H 3200 7450 50  0000 C CNN
-F 2 "" H 3200 7300 50  0000 C CNN
-F 3 "" H 3200 7300 50  0000 C CNN
-	1    3200 7300
-	1    0    0    -1
-$EndComp
-$Comp
-L VCC #PWR?
-U 1 1 57D1AD5D
-P 4200 7300
-F 0 "#PWR?" H 4200 7150 50  0001 C CNN
-F 1 "VCC" H 4200 7450 50  0000 C CNN
-F 2 "" H 4200 7300 50  0000 C CNN
-F 3 "" H 4200 7300 50  0000 C CNN
-	1    4200 7300
-	1    0    0    -1
-$EndComp
-Text GLabel 1300 7600 2    50   Input ~ 0
-XMAX
-Text GLabel 2300 7600 2    50   Input ~ 0
-YMAX
-Text GLabel 3300 7600 2    50   Input ~ 0
-ZMAX
-Text GLabel 4300 7600 2    50   Input ~ 0
-EMAX
-Wire Wire Line
-	1100 7400 1200 7400
-Wire Wire Line
-	1200 7400 1200 7300
-Wire Wire Line
-	1100 7500 1200 7500
-Wire Wire Line
-	1200 7500 1200 7700
-Wire Wire Line
-	1100 7600 1300 7600
-Wire Wire Line
-	2100 7400 2200 7400
-Wire Wire Line
-	2200 7400 2200 7300
-Wire Wire Line
-	2100 7500 2200 7500
-Wire Wire Line
-	2200 7500 2200 7700
-Wire Wire Line
-	2100 7600 2300 7600
-Wire Wire Line
-	3100 7600 3300 7600
-Wire Wire Line
-	4100 7600 4300 7600
-Wire Wire Line
-	4200 7700 4200 7500
-Wire Wire Line
-	4200 7500 4100 7500
-Wire Wire Line
-	4100 7400 4200 7400
-Wire Wire Line
-	4200 7400 4200 7300
-Wire Wire Line
-	3200 7700 3200 7500
-Wire Wire Line
-	3200 7500 3100 7500
-Wire Wire Line
-	3100 7400 3200 7400
-Wire Wire Line
-	3200 7400 3200 7300
 $EndSCHEMATC
