File: FireMC-3.14.kicad_pcb (KiCad board)
At the start: 2 copper layers, 123 parts, among them J1 Header_1X2, J10 Header_2X3, J11 Header_2X3, J12 Header_1X3, J13 Header_1X2, J14 Header_1X3, J15 Header_1X2, J16 Header_1X3, J17 Header_2X20, J18 Header_1X3, J19 Header_1X2, J2 Header_1X2, J20 Header_1X4, J3 Header_1X4, J4 Header_1X4, J5 Header_1X2, J6 Header_2X3, J7 Header_2X3, J8 Header_1X4, J9 Header_1X4, Q1 STD86N3LH5, Q2 STD86N3LH5, Q3 STD86N3LH5, Q4 STD86N3LH5, Q5 STD86N3LH5, Q6 STD86N3LH5, Q7 STD86N3LH5, U1 ISL6420B, U2 ISL6420B, U3 TMC_SILENT_STEPSTICK, U4 TMC_SILENT_STEPSTICK, U5 74LVC1G14, U6 74LV32, U7 TMC_SILENT_STEPSTICK, U8 TMC_SILENT_STEPSTICK, U9 MCP23S17

Commit message: Time to Update.  Board layout started.
Parts:
- added MH1: MOUNT_PTH, IPC_MFG:IMELLC_PTH_2.75x6.00, F.Cu at (360.9, 189.5)
- added MH2: MOUNT_PTH, IPC_MFG:IMELLC_PTH_2.75x6.00, F.Cu at (388.9, 204.0)
- added MH3: MOUNT_PTH, IPC_MFG:IMELLC_PTH_2.75x6.00, F.Cu at (384.6, 185.2)
- added MH4: MOUNT_PTH, IPC_MFG:IMELLC_PTH_2.75x6.00, F.Cu at (409.2, 195.1)
- J17: footprint IPC_MFG:SULLINS_PPTC202LFBN-RC -> IPC_MFG:SULLINS_PPxC202LFBN-RC
- R20, R22, R25, R26, R27, R28: moved to B.Cu
- U5: value 74LVC1G14 -> TMC_SILENT_STEPSTICK; footprint IPC_SOT:SOT95P280X145-5N -> IPC_MFG:stepstick
- U6: value 74LV32 -> TMC_SILENT_STEPSTICK; footprint IPC_SOP:SOP65P640X120-14N -> IPC_MFG:stepstick
- U7: value TMC_SILENT_STEPSTICK -> 74LVC1G14; footprint IPC_MFG:stepstick -> IPC_SOT:SOT95P280X145-5N
- U8: value TMC_SILENT_STEPSTICK -> 74LV32; footprint IPC_MFG:stepstick -> IPC_SOP:SOP65P640X120-14N
- moved C12 270.6 mm to (141.2, 105.9), turned to 90 degrees
- moved C16 268.2 mm to (172.5, 112.3), turned to 90 degrees
- moved C13 262.3 mm to (134.4, 122.2)
- moved C17 260.1 mm to (179.8, 112.3), turned to 90 degrees
- moved R4 256.0 mm to (132.8, 126.2)
- moved C14 255.0 mm to (137.9, 125.7)
- moved R7 250.9 mm to (139.4, 119.1), turned to 180 degrees
- moved Q2 249.5 mm to (148.6, 115.5), turned to 270 degrees
- moved R5 248.2 mm to (139.4, 115.8), turned to 180 degrees
- moved U1 246.8 mm to (133.9, 108.5), turned to 180 degrees
- moved C15 245.4 mm to (137.2, 118.1), turned to 90 degrees
- moved C18 238.3 mm to (187.2, 112.3), turned to 90 degrees
- moved J4 229.6 mm to (198.6, 52.9)
- moved R6 229.2 mm to (139.4, 117.6), turned to 180 degrees
- moved Q1 223.3 mm to (148.6, 103.3), turned to 270 degrees
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Connections:
- net Net-(C1-Pad1) renamed /Power/12VIN
- net Net-(C16-Pad1) renamed /Power/3V3OUT
- net Net-(C34-Pad1) renamed /Power/5VOUT
- U5 pad 1: (no net) -> GND
- U5 pad 2: /Safety/ALLSTOP -> VCC
- U5 pad 3: GND -> Net-(J8-Pad1)
- U5 pad 4: ~ALLSTOP -> Net-(J8-Pad2)
- U5 pad 5: VCC -> Net-(J8-Pad3)
- U6 pad 1: EN1 -> GND
- U6 pad 10: ~ALLSTOP -> Net-(J11-Pad5)
- U6 pad 11: EN4_O -> Net-(J11-Pad3)
- U6 pad 12: EN4 -> Net-(J11-Pad1)
- U6 pad 13: ~ALLSTOP -> Net-(U6-Pad13)
- U6 pad 14: VCC -> Net-(U6-Pad13)
- U6 pad 2: ~ALLSTOP -> VCC
- U6 pad 3: EN1_O -> Net-(J9-Pad1)
- U6 pad 4: EN2 -> Net-(J9-Pad2)
- U6 pad 5: ~ALLSTOP -> Net-(J9-Pad3)
- U6 pad 6: EN2_O -> Net-(J9-Pad4)
- U6 pad 8: EN3_O -> +12V
- U6 pad 9: EN3 -> EN4_O
- U7 pad 1: GND -> (no net)
- U7 pad 2: VCC -> /Safety/ALLSTOP
- U7 pad 3: Net-(J8-Pad1) -> GND
- U7 pad 4: Net-(J8-Pad2) -> ~ALLSTOP
- U7 pad 5: Net-(J8-Pad3) -> VCC
- U8 pad 1: GND -> EN1
- U8 pad 10: Net-(J11-Pad5) -> ~ALLSTOP
- U8 pad 11: Net-(J11-Pad3) -> EN4_O
- U8 pad 12: Net-(J11-Pad1) -> EN4
- U8 pad 13: Net-(U8-Pad13) -> ~ALLSTOP
- U8 pad 14: Net-(U8-Pad13) -> VCC
- U8 pad 2: VCC -> ~ALLSTOP
- U8 pad 3: Net-(J9-Pad1) -> EN1_O
- U8 pad 4: Net-(J9-Pad2) -> EN2
- U8 pad 5: Net-(J9-Pad3) -> ~ALLSTOP
- U8 pad 6: Net-(J9-Pad4) -> EN2_O
- U8 pad 8: +12V -> EN3_O
- U8 pad 9: EN4_O -> EN3
