File: FireMC-3.14.kicad_pcb (KiCad board)
At the start: 2 copper layers, 112 x 88.5 mm, 131 parts, among them J1 Header_1X2, J10 Header_2X3, J11 Header_2X3, J12 Header_1X3, J13 Header_1X2, J14 Header_1X3, J15 Header_1X2, J16 Header_1X3, J17 Header_2X20, J18 Header_1X3, J19 Header_1X2, J2 Header_1X2, J20 Header_1X4, J3 Header_1X4, J4 Header_1X4, J5 Header_1X2, J6 Header_2X3, J7 Header_2X3, J8 Header_1X4, J9 Header_1X4, Q1 STD86N3LH5, Q2 STD86N3LH5, Q3 STD86N3LH5, Q4 STD86N3LH5, Q5 STD86N3LH5, Q6 STD86N3LH5, Q7 STD86N3LH5, U1 ISL6420B, U2 ISL6420B, U3 TMC_SILENT_STEPSTICK, U4 TMC_SILENT_STEPSTICK, U5 TMC_SILENT_STEPSTICK, U6 TMC_SILENT_STEPSTICK, U7 74LVC1G14, U8 74LV32, U9 MCP23S17

Commit message: Changed Power management
Parts:
- removed C26, C39: 2u2, IPC_CAP:CAPC1608X90N
- removed C27: 10n, IPC_CAP:CAPC1608X90N
- removed C28, C29: 0u1, IPC_CAP:CAPC1608X90N
- removed C30: 220n, IPC_CAP:CAPC1608X90N
- removed C31: 62p, IPC_CAP:CAPC1608X90N
- removed C32: 1n5, IPC_CAP:CAPC1608X90N
- removed C33: 6n2, IPC_CAP:CAPC1608X90N
- removed C34, C35, C36: 150u, IPC_CAP:CAPAE660X770N
- removed C37, C38, C40, C41: 100u, IPC_CAP:CAPAE840X650N
- removed C5: 10u, IPC_CAP:CAPC1608X95N
- removed D5: LED, IPC_LED:LEDM1608X70N
- removed F3: 5A, IPC_MFG:MPD_BK-6010
- removed L2: 8u2, IPC_IND:INDM1213X620N
- removed R32, R33: 3k3, IPC_RES:RESC1608X55N
- removed R34, R35, R36: 2k21, IPC_RES:RESC1608X55N
- C12: value 180n -> 220n
- C19, C20: value 10u -> 1u; footprint IPC_CAP:CAPC1608X95N -> IPC_CAP:CAPC1608X90N
- C21, C22, C23: value 10u -> 100u; footprint IPC_CAP:CAPC1608X95N -> IPC_CAP:CAPAE840X650N
- C24: value 4u7 -> 100u; footprint IPC_CAP:CAPC1608X95N -> IPC_CAP:CAPAE840X650N
- C25: value 0u1 -> 2u2
- C6, C7: moved to B.Cu
- D2: value PMEG3050EP,115 -> LED; footprint IPC_SOD:SOD4725X100N -> IPC_LED:LEDM1608X70N
- J10, J11: value Header_2X3 -> Header_1X3; footprint IPC_MFG:TE_5-146254-3 -> IPC_MFG:SULLINS_PRPC003SAAN-RC
- J12, J16: value Header_1X3 -> Header_1X4; footprint IPC_MFG:SULLINS_PRPC003SAAN-RC -> IPC_MFG:SULLINS_PRPC004SAAN-RC
- J13: value Header_1X2 -> Header_1X4; footprint IPC_MFG:SULLINS_PRPC002SAAN-RC -> IPC_MFG:SULLINS_PRPC004SAAN-RC
- J14, J18: value Header_1X3 -> Header_2X3; footprint IPC_MFG:SULLINS_PRPC003SAAN-RC -> IPC_MFG:TE_5-146254-3
- J15, J19: value Header_1X2 -> Header_2X3; footprint IPC_MFG:SULLINS_PRPC002SAAN-RC -> IPC_MFG:TE_5-146254-3
- J17: value Header_2X20 -> Header_1X4; footprint IPC_MFG:SULLINS_PPTC202LFBN-RC -> IPC_MFG:SULLINS_PRPC004SAAN-RC
- J20: value Header_1X4 -> Header_1X2; footprint IPC_MFG:MOLEX_22-23-2041 -> IPC_MFG:SULLINS_PRPC002SAAN-RC
- J3: footprint IPC_MFG:SULLINS_PRPC004SAAN-RC -> IPC_MFG:MOLEX_22-23-2041
- J4: value Header_1X4 -> Header_2X20; footprint IPC_MFG:SULLINS_PRPC004SAAN-RC -> IPC_MFG:SULLINS_PPTC202LFBN-RC
- J6, J7: value Header_2X3 -> Header_1X2; footprint IPC_MFG:TE_5-146254-3 -> IPC_MFG:SULLINS_PRPC002SAAN-RC
- J8, J9: value Header_1X4 -> Header_1X3; footprint IPC_MFG:SULLINS_PRPC004SAAN-RC -> IPC_MFG:SULLINS_PRPC003SAAN-RC
- Q1, Q2: value STD86N3LH5 -> SI7386DP; footprint IPC_TO:TO228P972X240-3N -> IPC_SON:SON9P127_490X590X112L61X41T376X348N
- Q3, Q4: value STD86N3LH5 -> RE1J002YNTCL; footprint IPC_TO:TO228P972X240-3N -> IPC_SOFL:SOTFL3P50_160X85L45X28N
- R10: value 510R -> 2k21
- R11: value 56k2 -> 2k21
- R12: value 1k37 -> 2k21
- R13: value 10k -> 3k3
- R14: value 178R -> 3k3
- R15: value 330R -> 3k3
- R19, R25: value 100k -> 3k3
- R2: value 2k5 -> 1k
- R23, R29: value 3k3 -> 100k
- R3: value 499R -> 665R
- R31: value 3k3 -> 330R
- R4: value 56k2 -> 10k
- R5: value 2k21 -> 1k37
- R6: value 10k -> 191R
- R7: value 196R -> 56k2
- R9: value 1k -> 10k
- U1: value ISL6420B -> ISL6420BIRZ; footprint IPC_SOP:SOP63P600X155-20N -> IPC_QFN:QFN21P50_400X400X100L55X24T210N
- U2: value ISL6420B -> LP38693SD; footprint IPC_SOP:SOP63P600X155-20N -> IPC_SON:SON7P95_300X300X80L40X35T210X160N
- U3: value TMC_SILENT_STEPSTICK -> MCP23S17; footprint IPC_MFG:stepstick -> IPC_SOIC127P:SOIC127P1030X265-28N
- U7: value 74LVC1G14 -> TMC_SILENT_STEPSTICK; footprint IPC_SOT:SOT95P280X145-5N -> IPC_MFG:stepstick
- U9: value MCP23S17 -> 74LVC1G14; footprint IPC_SOIC127P:SOIC127P1030X265-28N -> IPC_SOT:SOT95P280X145-5N
- moved Q2 212.3 mm to (109.0, 243.5)
- moved R31 188.0 mm to (367.0, 186.4)
- moved Q1 185.9 mm to (125.9, 228.9)
- moved D1 185.3 mm to (96.4, 238.2)
- moved J17 184.9 mm to (245.4, 212.3)
- moved U9 182.8 mm to (361.1, 195.2)
- moved R30 179.4 mm to (353.6, 206.6)
- moved MH6 178.2 mm to (186.5, 82.5)
- moved C13 175.7 mm to (127.2, 245.1)
- moved C10 170.8 mm to (123.7, 245.1)
- moved R6 170.3 mm to (136.4, 245.3)
- moved C11 165.9 mm to (146.8, 227.2), turned to 0 degrees
- moved C12 165.3 mm to (132.1, 240.9)
- moved R2 164.2 mm to (145.8, 237.4)
- moved C17 163.7 mm to (125.0, 236.9)
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Connections:
- C10 pad 1: Net-(C10-Pad1) -> /Power/DLY
- C11 pad 2: Net-(C11-Pad2) -> /Power/OVP
- C12 pad 1: Net-(C12-Pad1) -> /Power/PH
- C12 pad 2: Net-(C12-Pad2) -> /Power/BOOT
- C13 pad 1: Net-(C13-Pad1) -> /Power/FB
- C13 pad 2: Net-(C13-Pad2) -> /Power/COMP
- C14 pad 1: Net-(C14-Pad1) -> /Power/Z1
- C14 pad 2: Net-(C13-Pad2) -> /Power/COMP
- C15 pad 1: Net-(C15-Pad1) -> /Power/Z2
- C15 pad 2: Net-(C13-Pad1) -> /Power/FB
- C16 pad 1: /Power/3V3OUT -> /Power/5VOUT
- C17 pad 1: /Power/3V3OUT -> /Power/5VOUT
- C18 pad 1: /Power/3V3OUT -> /Power/5VOUT
- C19 pad 1: /Power/12VIN -> +5V
- C20 pad 1: /Power/12VIN -> VCC
- C21 pad 1: /Power/12VIN -> +12V
- C22 pad 1: /Power/12VIN -> +12V
- C23 pad 1: /Power/12VIN -> +12V
- C24 pad 1: Net-(C24-Pad1) -> +12V
- C25 pad 1: Net-(C24-Pad1) -> /Safety/ALLSTOP
- C6 pad 1: Net-(C6-Pad1) -> /Power/VCC5
- C7 pad 1: Net-(C6-Pad1) -> /Power/VCC5
- C8 pad 1: Net-(C8-Pad1) -> /Power/REF
- C9 pad 1: Net-(C9-Pad1) -> /Power/EN
- D1 pad 1: Net-(C12-Pad2) -> /Power/BOOT
- D1 pad 2: Net-(C6-Pad1) -> /Power/VCC5
- D2 pad 1: Net-(C30-Pad2) -> Net-(D2-Pad1)
- D2 pad 2: Net-(C24-Pad1) -> +12V
- J10 pad 1: Net-(J10-Pad1) -> VCC
- J10 pad 2: VCC -> GND
- J10 pad 3: Net-(J10-Pad3) -> ZMAX
- J11 pad 1: Net-(J11-Pad1) -> VCC
- J11 pad 2: VCC -> GND
- J11 pad 3: Net-(J11-Pad3) -> EMAX
- J12 pad 1: VCC -> Net-(J12-Pad1)
- J12 pad 2: GND -> Net-(J12-Pad2)
- J12 pad 3: XMAX -> Net-(J12-Pad3)
- J13 pad 1: VCC -> Net-(J13-Pad1)
- J14 pad 1: VCC -> Net-(J14-Pad1)
- J14 pad 2: GND -> VCC
- J14 pad 3: YMAX -> Net-(J14-Pad3)
- J15 pad 1: VCC -> Net-(J15-Pad1)
- J15 pad 2: Net-(J15-Pad2) -> VCC
- J16 pad 1: VCC -> Net-(J16-Pad1)
- J16 pad 2: GND -> Net-(J16-Pad2)
- J16 pad 3: ZMAX -> Net-(J16-Pad3)
- J17 pad 3: SDA1 -> Net-(J17-Pad3)
- J18 pad 1: VCC -> Net-(J18-Pad1)
- J18 pad 2: GND -> VCC
- J18 pad 3: EMAX -> Net-(J18-Pad3)
- J19 pad 1: VCC -> Net-(J19-Pad1)
- J19 pad 2: Net-(J19-Pad2) -> VCC
- J20 pad 1: +5V -> Net-(J20-Pad1)
- J20 pad 2: Net-(J20-Pad2) -> GND
- J3 pad 1: Net-(J3-Pad1) -> +5V
- J3 pad 4: Net-(J3-Pad4) -> GND
- J4 pad 3: Net-(J4-Pad3) -> SDA1
- J5 pad 1: Net-(J5-Pad1) -> VCC
- J5 pad 2: GND -> Net-(J5-Pad2)
- J6 pad 1: Net-(J6-Pad1) -> VCC
- J6 pad 2: VCC -> Net-(J6-Pad2)
- J7 pad 1: Net-(J7-Pad1) -> VCC
- J7 pad 2: VCC -> Net-(J7-Pad2)
- J8 pad 1: Net-(J8-Pad1) -> VCC
- J8 pad 2: Net-(J8-Pad2) -> GND
- J8 pad 3: Net-(J8-Pad3) -> XMAX
- J9 pad 1: Net-(J9-Pad1) -> VCC
- J9 pad 2: Net-(J9-Pad2) -> GND
- J9 pad 3: Net-(J9-Pad3) -> YMAX
- L1 pad 1: Net-(C12-Pad1) -> /Power/PH
- L1 pad 2: /Power/3V3OUT -> /Power/5VOUT
- Q1 pad 1: Net-(Q1-Pad1) -> /Power/12VIN
- Q1 pad 3: Net-(C12-Pad1) -> /Power/12VIN
- Q2 pad 1: Net-(Q2-Pad1) -> /Power/PH
- Q2 pad 2: Net-(C12-Pad1) -> /Power/PH
- Q2 pad 3: GND -> /Power/PH
- Q3 pad 1: Net-(Q3-Pad1) -> VCC
- Q3 pad 2: /Power/12VIN -> GND
- Q3 pad 3: Net-(C30-Pad1) -> /Power/PGD3
- Q4 pad 1: Net-(Q4-Pad1) -> PG5
- Q4 pad 2: Net-(C30-Pad1) -> GND
- Q4 pad 3: GND -> /Power/PGD5
- Q5 pad 2: Net-(J13-Pad2) -> Net-(J5-Pad2)
- Q6 pad 2: Net-(J15-Pad2) -> Net-(J6-Pad2)
- Q7 pad 2: Net-(J19-Pad2) -> Net-(J7-Pad2)
- R1 pad 1: +5V -> /Power/12VIN
- R1 pad 2: Net-(C9-Pad1) -> /Power/EN
- R10 pad 1: /Power/12VIN -> Net-(D2-Pad1)
- R10 pad 2: Net-(C29-Pad2) -> GND
- R11 pad 1: Net-(C31-Pad1) -> Net-(D3-Pad1)
- R11 pad 2: Net-(C32-Pad1) -> /Power/PGD5
- R12 pad 1: GND -> Net-(D4-Pad1)
- R12 pad 2: Net-(C31-Pad1) -> /Power/PGD3
- R13 pad 1: /Power/5VOUT -> VCC
- R13 pad 2: Net-(C31-Pad1) -> SPI_CE0
- R14 pad 1: /Power/5VOUT -> VCC
- R14 pad 2: Net-(C33-Pad1) -> Net-(R14-Pad2)
- R15 pad 1: /Safety/ALLSTOP -> PMP
- R15 pad 2: Net-(J5-Pad1) -> GND
- R16 pad 1: VCC -> VLV
- R16 pad 2: /Safety/ALLSTOP -> GND
- R17 pad 1: VCC -> AUX
- R17 pad 2: EN1_O -> GND
- R18 pad 2: EN2_O -> EN1_O
- R19 pad 1: Net-(J6-Pad1) -> VCC
- R19 pad 2: GND -> EN3_O
- R2 pad 1: Net-(C9-Pad1) -> /Power/EN
- R20 pad 1: Net-(J7-Pad1) -> Net-(J14-Pad1)
- R21 pad 1: Net-(J6-Pad5) -> Net-(J14-Pad5)
- R22 pad 1: Net-(J7-Pad5) -> Net-(J15-Pad1)
- R23 pad 1: VCC -> Net-(J15-Pad5)
- R23 pad 2: EN3_O -> GND
- R24 pad 2: EN4_O -> EN2_O
- R25 pad 1: Net-(J10-Pad1) -> VCC
- R25 pad 2: GND -> EN4_O
- R26 pad 1: Net-(J11-Pad1) -> Net-(J18-Pad1)
- R27 pad 1: Net-(J10-Pad5) -> Net-(J18-Pad5)
- R28 pad 1: Net-(J11-Pad5) -> Net-(J19-Pad1)
- R29 pad 1: PMP -> Net-(J19-Pad5)
- R3 pad 2: Net-(C11-Pad2) -> /Power/OVP
- R30 pad 1: VLV -> VCC
- R30 pad 2: GND -> /Safety/ALLSTOP
- R31 pad 1: AUX -> /Safety/ALLSTOP
- R31 pad 2: GND -> Net-(J20-Pad1)
- R4 pad 1: Net-(C13-Pad1) -> /Power/5VOUT
- R4 pad 2: Net-(C14-Pad1) -> /Power/FB
- R5 pad 2: Net-(C13-Pad1) -> /Power/FB
- R6 pad 1: /Power/3V3OUT -> /Power/5VOUT
- R6 pad 2: Net-(C13-Pad1) -> /Power/Z2
- R7 pad 1: /Power/3V3OUT -> /Power/FB
- R7 pad 2: Net-(C15-Pad1) -> /Power/Z1
- R8 pad 1: /Power/12VIN -> +12V
- R8 pad 2: Net-(C27-Pad1) -> /Power/PGD5
- R9 pad 1: Net-(C27-Pad1) -> +12V
- R9 pad 2: GND -> /Power/PGD3
- U1 pad 1: Net-(C10-Pad1) -> GND
- U1 pad 10: Net-(C11-Pad2) -> /Power/FB
- U1 pad 11: Net-(C8-Pad1) -> /Power/COMP
- U1 pad 12: GND -> /Power/EN
- U1 pad 13: Net-(C6-Pad1) -> PG5
- U1 pad 14: /Power/12VIN -> /Power/DLY
- U1 pad 16: Net-(C6-Pad1) -> /Power/LG
- U1 pad 17: Net-(C13-Pad1) -> /Power/VCC5
- U1 pad 18: Net-(C13-Pad2) -> /Power/PH
- U1 pad 19: Net-(C9-Pad1) -> /Power/UG
- U1 pad 20: PGD3 -> /Power/BOOT
- U1 pad 3: Net-(Q2-Pad1) -> /Power/OVP
- U1 pad 4: Net-(C6-Pad1) -> /Power/REF
- U1 pad 5: Net-(C12-Pad1) -> GND
- U1 pad 6: Net-(Q1-Pad1) -> /Power/VCC5
- U1 pad 7: Net-(C12-Pad2) -> /Power/12VIN
- U1 pad 9: GND -> /Power/VCC5
- U2 pad 1: Net-(C28-Pad1) -> +5V
- U2 pad 3: Net-(Q4-Pad1) -> +5V
- U2 pad 4: Net-(C24-Pad1) -> VCC
- U2 pad 5: Net-(C30-Pad1) -> VCC
- U2 pad 6: Net-(Q3-Pad1) -> +5V
- U2 pad 7: Net-(C30-Pad2) -> GND
- U3 pad 1: GND -> Net-(U3-Pad1)
- U3 pad 10: Net-(J6-Pad5) -> GND
- U3 pad 11: Net-(J6-Pad3) -> SPI_CE0
- U3 pad 12: Net-(J6-Pad1) -> SPI_SLCK
- U3 pad 13: Net-(U3-Pad13) -> SPI_MOSI
- U3 pad 14: Net-(U3-Pad13) -> SPI_MISO
- U3 pad 15: STEP1 -> GND
- U3 pad 16: DIR1 -> GND
- U3 pad 2: VCC -> Net-(U3-Pad2)
- U3 pad 3: Net-(J3-Pad1) -> Net-(U3-Pad3)
- U3 pad 4: Net-(J3-Pad2) -> Net-(U3-Pad4)
- U3 pad 5: Net-(J3-Pad3) -> Net-(U3-Pad5)
- U3 pad 6: Net-(J3-Pad4) -> Net-(U3-Pad6)
- U3 pad 7: GND -> Net-(U3-Pad7)
- U3 pad 8: +12V -> Net-(U3-Pad8)
- U3 pad 9: EN1_O -> VCC
- U4 pad 10: Net-(J7-Pad5) -> Net-(J14-Pad5)
- U4 pad 11: Net-(J7-Pad3) -> Net-(J14-Pad3)
- U4 pad 12: Net-(J7-Pad1) -> Net-(J14-Pad1)
- U4 pad 15: STEP2 -> STEP1
- U4 pad 16: DIR2 -> DIR1
- U4 pad 3: Net-(J4-Pad1) -> Net-(J12-Pad1)
- U4 pad 4: Net-(J4-Pad2) -> Net-(J12-Pad2)
- U4 pad 5: Net-(J4-Pad3) -> Net-(J12-Pad3)
- U4 pad 6: Net-(J4-Pad4) -> Net-(J12-Pad4)
- U4 pad 9: EN2_O -> EN1_O
- U5 pad 10: Net-(J10-Pad5) -> Net-(J15-Pad5)
- U5 pad 11: Net-(J10-Pad3) -> Net-(J15-Pad3)
- U5 pad 12: Net-(J10-Pad1) -> Net-(J15-Pad1)
- U5 pad 3: Net-(J8-Pad1) -> Net-(J13-Pad1)
- U5 pad 4: Net-(J8-Pad2) -> Net-(J13-Pad2)
- U5 pad 5: Net-(J8-Pad3) -> Net-(J13-Pad3)
- U5 pad 6: Net-(J8-Pad4) -> Net-(J13-Pad4)
- U6 pad 10: Net-(J11-Pad5) -> Net-(J18-Pad5)
- U6 pad 11: Net-(J11-Pad3) -> Net-(J18-Pad3)
- U6 pad 12: Net-(J11-Pad1) -> Net-(J18-Pad1)
- U6 pad 15: STEP4 -> STEP2
- U6 pad 16: DIR4 -> DIR2
- U6 pad 3: Net-(J9-Pad1) -> Net-(J16-Pad1)
- U6 pad 4: Net-(J9-Pad2) -> Net-(J16-Pad2)
- U6 pad 5: Net-(J9-Pad3) -> Net-(J16-Pad3)
- U6 pad 6: Net-(J9-Pad4) -> Net-(J16-Pad4)
- U6 pad 9: EN4_O -> EN2_O
- U7 pad 1: (no net) -> GND
- U7 pad 2: /Safety/ALLSTOP -> VCC
- U7 pad 3: GND -> Net-(J17-Pad1)
- U7 pad 4: ~ALLSTOP -> Net-(J17-Pad2)
- U7 pad 5: VCC -> Net-(J17-Pad3)
- U9 pad 1: Net-(U9-Pad1) -> (no net)
- U9 pad 2: Net-(U9-Pad2) -> /Safety/ALLSTOP
- U9 pad 3: Net-(U9-Pad3) -> GND
- U9 pad 4: Net-(U9-Pad4) -> ~ALLSTOP
- U9 pad 5: Net-(U9-Pad5) -> VCC
Routing:
- net /Power/VCC5: track 0.00 -> 12.7 mm, vias 0 -> 3
- net GND: track 0.00 -> 8.33 mm
Other:
- board size 112 x 88.5 mm -> 112 x 85 mm
- net class 12V added: clearance 0.127, trace_width 2.6, via_dia 0.6, via_drill 0.4
- net class 5V added: clearance 0.127, trace_width 2.794, via_dia 0.6, via_drill 0.4
- net class Default: clearance 0.2 -> 0.127; trace_width 0.25 -> 0.254
- rule trace_clearance: 0.2 -> 0.127

Commit message: Pre-reformat Backup
Parts:
- moved C10 108.2 mm to (137.3, 137.8), turned to 90 degrees
- moved D1 108.2 mm to (130.2, 135.4), turned to 180 degrees
- moved R2 96.6 mm to (139.2, 141.1), turned to 270 degrees
- moved C8 94.7 mm to (130.5, 141.1), turned to 270 degrees
- moved R1 92.6 mm to (137.6, 141.1), turned to 90 degrees
- moved R9 87.4 mm to (65.9, 211.9)
- moved R11 83.8 mm to (68.5, 216.5)
- moved C9 81.1 mm to (140.8, 141.1), turned to 270 degrees
- moved R12 80.1 mm to (66.9, 222.0)
- moved R10 78.1 mm to (72.8, 221.5)
- moved Q4 78.1 mm to (114.2, 156.9)
- moved R8 67.6 mm to (69.6, 227.4)
- moved Q3 54.6 mm to (108.5, 156.9)
- moved D3 33.4 mm to (80.5, 216.1)
- moved D2 23.7 mm to (80.5, 212.0)
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Routing:
- net /Power/EN: track 0.00 -> 5.76 mm

Commit message: update
Parts:
- U1: value ISL6420BIRZ -> ISL6420BIAZ; footprint IPC_QFN:QFN21P50_400X400X100L55X24T210N -> IPC_SOP:SOP63P600X155-20N
- moved Q2 128.0 mm to (138.0, 118.9), turned to 270 degrees
- moved R6 127.7 mm to (107.8, 120.9)
- moved R7 124.3 mm to (111.1, 119.3)
- moved R4 119.3 mm to (107.8, 119.3)
- moved R5 118.0 mm to (111.1, 117.6), turned to 180 degrees
- moved C15 115.4 mm to (109.5, 122.6)
- moved C12 112.5 mm to (95.9, 134.4), turned to 180 degrees
- moved C13 110.7 mm to (102.4, 137.3)
- moved R3 109.3 mm to (91.6, 139.8), turned to 90 degrees
- moved C14 107.0 mm to (112.0, 121.7), turned to 270 degrees
- moved Q1 105.3 mm to (93.1, 128.8), turned to 270 degrees
- moved C11 104.2 mm to (89.9, 139.8), turned to 90 degrees
- moved Q4 67.6 mm to (67.3, 205.6)
- moved Q3 59.5 mm to (74.0, 205.4)
- moved D1 37.6 mm to (92.6, 134.7), turned to 270 degrees
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Connections:
- net GPIO24 renamed Net-(J4-Pad18)
- net GPIO27 renamed Net-(J4-Pad13)
- net GPIO5 renamed Net-(J4-Pad29)
- net GPIO6 renamed Net-(J4-Pad31)
- net ID_SC renamed Net-(J4-Pad28)
- net ID_SD renamed Net-(J4-Pad27)
- net SCL1 renamed Net-(J4-Pad5)
- net SDA1 renamed Net-(J4-Pad3)
- net SPI_CE1 renamed Net-(J4-Pad26)
- J4 pad 22: GPIO25 -> Net-(J4-Pad22)
- J4 pad 37: GPIO25 -> Net-(J4-Pad37)
- U1 pad 1: GND -> /Power/DLY
- U1 pad 10: /Power/FB -> /Power/OVP
- U1 pad 11: /Power/COMP -> /Power/REF
- U1 pad 12: /Power/EN -> GND
- U1 pad 13: PG5 -> /Power/VCC5
- U1 pad 14: /Power/DLY -> /Power/12VIN
- U1 pad 16: /Power/LG -> /Power/VCC5
- U1 pad 17: /Power/VCC5 -> /Power/FB
- U1 pad 18: /Power/PH -> /Power/COMP
- U1 pad 19: /Power/UG -> /Power/EN
- U1 pad 20: /Power/BOOT -> PG5
- U1 pad 3: /Power/OVP -> /Power/LG
- U1 pad 4: /Power/REF -> /Power/VCC5
- U1 pad 5: GND -> /Power/PH
- U1 pad 6: /Power/VCC5 -> /Power/UG
- U1 pad 7: /Power/12VIN -> /Power/BOOT
- U1 pad 9: /Power/VCC5 -> GND
Routing:
- net /Power/VCC5: track 12.7 -> 1.90 mm, vias 3 -> 0
- net GND: track 8.33 -> 0.00 mm
- net /Power/EN: track 5.76 -> 4.19 mm
