File: FireMC-3.14_IO.sch (KiCad schematic (older format))
At the start: 18 parts, among them J12 Header_1X3, J13 Header_1X2, J14 Header_1X3, J15 Header_1X2, J16 Header_1X3, J17 Header_2X20, J18 Header_1X3, J19 Header_1X2, J20 Header_1X4, Q5 STD86N3LH5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

Commit message: Update 1/1/2017
Parts:
- J17: footprint IPC_MFG:SULLINS_PPxC202LFBN-RC -> IPC_MFG:SULLINS_PPTC202LFBN-RC
Changed lines of the file:
@@
 F 0 "J17" H 3350 3750 60  0000 C CNN
 F 1 "Header_2X20" H 3350 1550 60  0000 C CNN
-F 2 "IPC_MFG:SULLINS_PPxC202LFBN-RC" H 3350 2650 60  0001 C CNN
+F 2 "IPC_MFG:SULLINS_PPTC202LFBN-RC" H 3350 2650 60  0001 C CNN
 F 3 "" H 3350 2650 60  0000 C CNN
 F 4 "PPPC200LFBN-RC" H 3350 2650 60  0001 C CNN "Mfg PN"
