File: FireMC-3.14_IO.sch (KiCad schematic (older format))
At the start: 18 parts, among them J12 Header_1X3, J13 Header_1X2, J14 Header_1X3, J15 Header_1X2, J16 Header_1X3, J17 Header_2X20, J18 Header_1X3, J19 Header_1X2, J20 Header_1X4, Q5 STD86N3LH5, Q6 STD86N3LH5, Q7 STD86N3LH5, U9 MCP23S17

Commit message: Changed Power management
Parts:
- renumbered J16 to J10, J18 to J11, J20 to J3, J17 to J4, J13 to J5, J15 to J6, J19 to J7, J12 to J8, J14 to J9, R32 to R13, R33 to R14, R29 to R15, R30 to R16, R31 to R17, U9 to U3
Connections:
- net EXP_INTA: no longer names the net of U3.20 (INTA)
- net EXP_INTB: no longer names the net of U3.19 (INTB)
- no-connect marks 15 -> 17
Changed lines of the file:
@@
 LIBS:Intersil
 LIBS:mounting hole
+LIBS:TI
+LIBS:power_transistors
 LIBS:FireMC-3.14-cache
 EELAYER 25 0
@@
 $EndDescr
 $Comp
-L Header_2X20 J17
+L Header_2X20 J4
 U 1 1 57CB4A0A
 P 3350 2650
-F 0 "J17" H 3350 3750 60  0000 C CNN
+F 0 "J4" H 3350 3750 60  0000 C CNN
 F 1 "Header_2X20" H 3350 1550 60  0000 C CNN
 F 2 "IPC_MFG:SULLINS_PPTC202LFBN-RC" H 3350 2650 60  0001 C CNN
@@
 	2400 2800 3000 2800
 Wire Wire Line
-	2400 3000 3000 3000
-Wire Wire Line
-	2400 1800 3000 1800
-Wire Wire Line
 	2400 1900 3000 1900
 Wire Wire Line
-	3700 3000 4300 3000
-Wire Wire Line
 	3700 2900 4300 2900
 Wire Wire Line
 	3700 2800 4300 2800
 $Comp
-L GND #PWR08
+L GND #PWR015
 U 1 1 57CB4DBD
 P 2900 3700
-F 0 "#PWR08" H 2900 3450 50  0001 C CNN
+F 0 "#PWR015" H 2900 3450 50  0001 C CNN
 F 1 "GND" H 2900 3550 50  0000 C CNN
 F 2 "" H 2900 3700 50  0000 C CNN
@@
 $EndComp
 $Comp
-L GND #PWR09
+L GND #PWR016
 U 1 1 57CB4DD3
 P 3800 3700
-F 0 "#PWR09" H 3800 3450 50  0001 C CNN
+F 0 "#PWR016" H 3800 3450 50  0001 C CNN
 F 1 "GND" H 3800 3550 50  0000 C CNN
 F 2 "" H 3800 3700 50  0000 C CNN
@@
 	3700 2700 4300 2700
 $Comp
-L Header_1X4 J20
+L Header_1X4 J3
 U 1 1 57CB6877
 P 8800 1850
-F 0 "J20" H 8800 2150 60  0000 C CNN
+F 0 "J3" H 8800 2150 60  0000 C CNN
 F 1 "Header_1X4" H 8800 1550 60  0000 C CNN
 F 2 "IPC_MFG:MOLEX_22-23-2041" H 8800 1850 60  0001 C CNN
@@
 $EndComp
 $Comp
-L GND #PWR010
+L GND #PWR017
 U 1 1 57CB72B4
 P 8400 2100
-F 0 "#PWR010" H 8400 1850 50  0001 C CNN
+F 0 "#PWR017" H 8400 1850 50  0001 C CNN
 F 1 "GND" H 8400 1950 50  0000 C CNN
 F 2 "" H 8400 2100 50  0000 C CNN
@@
 $EndComp
 $Comp
-L +5V #PWR011
+L +5V #PWR018
 U 1 1 57CB7418
 P 8400 1600
-F 0 "#PWR011" H 8400 1450 50  0001 C CNN
+F 0 "#PWR018" H 8400 1450 50  0001 C CNN
 F 1 "+5V" H 8400 1740 50  0000 C CNN
 F 2 "" H 8400 1600 50  0000 C CNN
@@
 	8400 1700 8400 1600
 $Comp
-L Header_1X2 J13
+L Header_1X2 J5
 U 1 1 57D1D48D
 P 1200 4850
-F 0 "J13" H 1200 5050 60  0000 C CNN
+F 0 "J5" H 1200 5050 60  0000 C CNN
 F 1 "Header_1X2" H 1200 4650 60  0000 C CNN
 F 2 "IPC_MFG:SULLINS_PRPC002SAAN-RC" H 1200 4750 60  0001 C CNN
@@
 $EndComp
 $Comp
-L Header_1X3 J12
+L Header_1X3 J8
 U 1 1 57D1D4A8
 P 900 7450
-F 0 "J12" H 900 7700 60  0000 C CNN
+F 0 "J8" H 900 7700 60  0000 C CNN
 F 1 "Header_1X3" H 900 7200 60  0000 C CNN
 F 2 "IPC_MFG:SULLINS_PRPC003SAAN-RC" H 900 7400 60  0001 C CNN
@@
 $EndComp
 $Comp
-L Header_1X2 J15
+L Header_1X2 J6
 U 1 1 57D1D4C7
 P 2800 4850
-F 0 "J15" H 2800 5050 60  0000 C CNN
+F 0 "J6" H 2800 5050 60  0000 C CNN
 F 1 "Header_1X2" H 2800 4650 60  0000 C CNN
 F 2 "IPC_MFG:SULLINS_PRPC002SAAN-RC" H 2800 4750 60  0001 C CNN
@@
 $EndComp
 $Comp
-L Header_1X2 J19
+L Header_1X2 J7
 U 1 1 57D1D4FC
 P 4500 4850
-F 0 "J19" H 4500 5050 60  0000 C CNN
+F 0 "J7" H 4500 5050 60  0000 C CNN
 F 1 "Header_1X2" H 4500 4650 60  0000 C CNN
 F 2 "IPC_MFG:SULLINS_PRPC002SAAN-RC" H 4500 4750 60  0001 C CNN
@@
 $EndComp
 $Comp
-L Header_1X3 J14
+L Header_1X3 J9
 U 1 1 57D1D53A
 P 2000 7450
-F 0 "J14" H 2000 7700 60  0000 C CNN
+F 0 "J9" H 2000 7700 60  0000 C CNN
 F 1 "Header_1X3" H 2000 7200 60  0000 C CNN
 F 2 "IPC_MFG:SULLINS_PRPC003SAAN-RC" H 2000 7400 60  0001 C CNN
@@
 $EndComp
 $Comp
-L Header_1X3 J16
+L Header_1X3 J10
 U 1 1 57D1D577
 P 3100 7450
-F 0 "J16" H 3100 7700 60  0000 C CNN
+F 0 "J10" H 3100 7700 60  0000 C CNN
 F 1 "Header_1X3" H 3100 7200 60  0000 C CNN
 F 2 "IPC_MFG:SULLINS_PRPC003SAAN-RC" H 3100 7400 60  0001 C CNN
@@
 $EndComp
 $Comp
-L Header_1X3 J18
+L Header_1X3 J11
 U 1 1 57D1D5C9
 P 4200 7450
-F 0 "J18" H 4200 7700 60  0000 C CNN
+F 0 "J11" H 4200 7700 60  0000 C CNN
 F 1 "Header_1X3" H 4200 7200 60  0000 C CNN
 F 2 "IPC_MFG:SULLINS_PRPC003SAAN-RC" H 4200 7400 60  0001 C CNN
@@
 $EndComp
 $Comp
-L VCC #PWR012
+L VCC #PWR019
 U 1 1 57D1D60D
 P 1300 7250
-F 0 "#PWR012" H 1300 7100 50  0001 C CNN
+F 0 "#PWR019" H 1300 7100 50  0001 C CNN
 F 1 "VCC" H 1300 7400 50  0000 C CNN
 F 2 "" H 1300 7250 50  0000 C CNN
@@
 $EndComp
 $Comp
-L VCC #PWR013
+L VCC #PWR020
 U 1 1 57D1D63A
 P 3500 7250
-F 0 "#PWR013" H 3500 7100 50  0001 C CNN
+F 0 "#PWR020" H 3500 7100 50  0001 C CNN
 F 1 "VCC" H 3500 7400 50  0000 C CNN
 F 2 "" H 3500 7250 50  0000 C CNN
@@
 $EndComp
 $Comp
-L VCC #PWR014
+L VCC #PWR021
 U 1 1 57D1D660
 P 4900 4700
-F 0 "#PWR014" H 4900 4550 50  0001 C CNN
+F 0 "#PWR021" H 4900 4550 50  0001 C CNN
 F 1 "VCC" H 4900 4850 50  0000 C CNN
 F 2 "" H 4900 4700 50  0000 C CNN
@@
 $EndComp
 $Comp
-L VCC #PWR015
+L VCC #PWR022
 U 1 1 57D1D686
 P 4600 7250
-F 0 "#PWR015" H 4600 7100 50  0001 C CNN
+F 0 "#PWR022" H 4600 7100 50  0001 C CNN
 F 1 "VCC" H 4600 7400 50  0000 C CNN
 F 2 "" H 4600 7250 50  0000 C CNN
@@
 $EndComp
 $Comp
-L GND #PWR016
+L GND #PWR023
 U 1 1 57D1D6AC
 P 1300 7650
-F 0 "#PWR016" H 1300 7400 50  0001 C CNN
+F 0 "#PWR023" H 1300 7400 50  0001 C CNN
 F 1 "GND" H 1300 7500 50  0000 C CNN
 F 2 "" H 1300 7650 50  0000 C CNN
@@
 $EndComp
 $Comp
-L GND #PWR017
+L GND #PWR024
 U 1 1 57D1D6D2
 P 1600 5800
-F 0 "#PWR017" H 1600 5550 50  0001 C CNN
+F 0 "#PWR024" H 1600 5550 50  0001 C CNN
 F 1 "GND" H 1600 5650 50  0000 C CNN
 F 2 "" H 1600 5800 50  0000 C CNN
@@
 $EndComp
 $Comp
-L GND #PWR018
+L GND #PWR025
 U 1 1 57D1D6F8
 P 3200 5800
-F 0 "#PWR018" H 3200 5550 50  0001 C CNN
+F 0 "#PWR025" H 3200 5550 50  0001 C CNN
 F 1 "GND" H 3200 5650 50  0000 C CNN
 F 2 "" H 3200 5800 50  0000 C CNN
@@
 $EndComp
 $Comp
-L GND #PWR019
+L GND #PWR026
 U 1 1 57D1D71E
 P 4900 5800
-F 0 "#PWR019" H 4900 5550 50  0001 C CNN
+F 0 "#PWR026" H 4900 5550 50  0001 C CNN
 F 1 "GND" H 4900 5650 50  0000 C CNN
 F 2 "" H 4900 5800 50  0000 C CNN
@@
 $EndComp
 $Comp
-L GND #PWR020
+L GND #PWR027
 U 1 1 57D1D744
 P 4600 7650
-F 0 "#PWR020" H 4600 7400 50  0001 C CNN
+F 0 "#PWR027" H 4600 7400 50  0001 C CNN
 F 1 "GND" H 4600 7500 50  0000 C CNN
 F 2 "" H 4600 7650 50  0000 C CNN
@@
 $EndComp
 $Comp
-L MCP23S17 U9
+L MCP23S17 U3
 U 1 1 57D1D763
 P 8900 5200
-F 0 "U9" H 9150 6150 50  0000 R CNN
+F 0 "U3" H 9150 6150 50  0000 R CNN
 F 1 "MCP23S17" H 8900 4250 50  0000 C CNN
 F 2 "IPC_SOIC127P:SOIC127P1030X265-28N" H 8450 4550 50  0001 C CNN
@@
 $EndComp
 $Comp
-L VCC #PWR021
+L VCC #PWR028
 U 1 1 57D1D96E
 P 7700 4300
-F 0 "#PWR021" H 7700 4150 50  0001 C CNN
+F 0 "#PWR028" H 7700 4150 50  0001 C CNN
 F 1 "VCC" H 7700 4450 50  0000 C CNN
 F 2 "" H 7700 4300 50  0000 C CNN
@@
 $EndComp
 $Comp
-L GND #PWR022
+L GND #PWR029
 U 1 1 57D1D997
 P 8300 6100
-F 0 "#PWR022" H 8300 5850 50  0001 C CNN
+F 0 "#PWR029" H 8300 5850 50  0001 C CNN
 F 1 "GND" H 8300 5950 50  0000 C CNN
 F 2 "" H 8300 6100 50  0000 C CNN
@@
 	1300 7350 1300 7250
 $Comp
-L VCC #PWR023
+L VCC #PWR030
 U 1 1 57D1DEB5
 P 2400 7250
-F 0 "#PWR023" H 2400 7100 50  0001 C CNN
+F 0 "#PWR030" H 2400 7100 50  0001 C CNN
 F 1 "VCC" H 2400 7400 50  0000 C CNN
 F 2 "" H 2400 7250 50  0000 C CNN
@@
 $EndComp
 $Comp
-L VCC #PWR024
+L VCC #PWR031
 U 1 1 57D1DEDE
 P 3200 4700
-F 0 "#PWR024" H 3200 4550 50  0001 C CNN
+F 0 "#PWR031" H 3200 4550 50  0001 C CNN
 F 1 "VCC" H 3200 4850 50  0000 C CNN
 F 2 "" H 3200 4700 50  0000 C CNN
@@
 $EndComp
 $Comp
-L VCC #PWR025
+L VCC #PWR032
 U 1 1 57D1DF07
 P 1600 4700
-F 0 "#PWR025" H 1600 4550 50  0001 C CNN
+F 0 "#PWR032" H 1600 4550 50  0001 C CNN
 F 1 "VCC" H 1600 4850 50  0000 C CNN
 F 2 "" H 1600 4700 50  0000 C CNN
@@
 $EndComp
 $Comp
-L GND #PWR026
+L GND #PWR033
 U 1 1 57D1DF30
 P 3500 7650
-F 0 "#PWR026" H 3500 7400 50  0001 C CNN
+F 0 "#PWR033" H 3500 7400 50  0001 C CNN
 F 1 "GND" H 3500 7500 50  0000 C CNN
 F 2 "" H 3500 7650 50  0000 C CNN
@@
 $EndComp
 $Comp
-L GND #PWR027
+L GND #PWR034
 U 1 1 57D1DF59
 P 2400 7650
-F 0 "#PWR027" H 2400 7400 50  0001 C CNN
+F 0 "#PWR034" H 2400 7400 50  0001 C CNN
 F 1 "GND" H 2400 7500 50  0000 C CNN
 F 2 "" H 2400 7650 50  0000 C CNN
@@
 SPI_MISO
 $Comp
-L R R32
+L R R13
 U 1 1 57D550E4
 P 7700 4650
-F 0 "R32" V 7780 4650 50  0000 C CNN
+F 0 "R13" V 7780 4650 50  0000 C CNN
 F 1 "3k3" V 7700 4650 50  0000 C CNN
 F 2 "IPC_RES:RESC1608X55N" V 7630 4650 50  0001 C CNN
@@
 	7700 4400 8400 4400
 $Comp
-L R R33
+L R R14
 U 1 1 57D55D38
 P 8000 4650
-F 0 "R33" V 8080 4650 50  0000 C CNN
+F 0 "R14" V 8080 4650 50  0000 C CNN
 F 1 "3k3" V 8000 4650 50  0000 C CNN
 F 2 "IPC_RES:RESC1608X55N" V 7930 4650 50  0001 C CNN
@@
 Wire Wire Line
 	8000 5500 8400 5500
-Text GLabel 7600 5700 0    50   Input ~ 0
-EXP_INTA
-Text GLabel 7600 5800 0    50   Input ~ 0
-EXP_INTB
-Wire Wire Line
-	7600 5700 8400 5700
-Wire Wire Line
-	8400 5800 7600 5800
 Text GLabel 9600 4600 2    50   Input ~ 0
 AUX
@@
 NoConn ~ 9400 6000
 $Comp
-L R R31
+L R R17
 U 1 1 57D58CCB
 P 5300 5450
-F 0 "R31" V 5380 5450 50  0000 C CNN
+F 0 "R17" V 5380 5450 50  0000 C CNN
 F 1 "3k3" V 5300 5450 50  0000 C CNN
 F 2 "IPC_RES:RESC1608X55N" V 5230 5450 50  0001 C CNN
@@
 $EndComp
 $Comp
-L R R30
+L R R16
 U 1 1 57D58E2F
 P 3600 5450
-F 0 "R30" V 3680 5450 50  0000 C CNN
+F 0 "R16" V 3680 5450 50  0000 C CNN
 F 1 "3k3" V 3600 5450 50  0000 C CNN
 F 2 "IPC_RES:RESC1608X55N" V 3530 5450 50  0001 C CNN
@@
 $EndComp
 $Comp
-L R R29
+L R R15
 U 1 1 57D58EA6
 P 2000 5450
-F 0 "R29" V 2080 5450 50  0000 C CNN
+F 0 "R15" V 2080 5450 50  0000 C CNN
 F 1 "3k3" V 2000 5450 50  0000 C CNN
 F 2 "IPC_RES:RESC1608X55N" V 1930 5450 50  0001 C CNN
@@
 Text Notes 4950 2450 2    50   ~ 0
 GPIO23
+NoConn ~ 8400 5700
+NoConn ~ 8400 5800
+Wire Wire Line
+	2400 3000 3000 3000
+Wire Wire Line
+	3700 3000 4300 3000
+Wire Wire Line
+	2400 1800 3000 1800
 $EndSCHEMATC

Commit message: KiCAD 4.0.5 Update corrections
Parts:
- removed U3: MCP23S17, IPC_SOIC127P:SOIC127P1030X265-28N, symbol MCP23S17
- added U?: MCP23S17, symbol MCP23S17
Connections:
- net AUX: now also U?.23 (GPA2)
- net EN1: now also U?.24 (GPA3)
- net EN2: now also U?.25 (GPA4)
- net EN3: now also U?.26 (GPA5)
- net EN4: now also U?.27 (GPA6)
- net GND: now also U?.10 (VSS), U?.15 (A0), U?.16 (A1), U?.17 (A2)
- net PMP: now also U?.21 (GPA0)
- net SPI_CE0: now also U?.11 (~CS)
- net SPI_MISO: now also U?.14 (SO)
- net SPI_MOSI: now also U?.13 (SI)
- net SPI_SLCK: now also U?.12 (SCK)
- net VCC: now also U?.9 (VDD)
- net VLV: now also U?.22 (GPA1)
- net at R14.2: now also U?.18 (~RST)
Changed lines of the file:
@@
 LIBS:microcontrollers
 LIBS:dsp
-LIBS:microchip
+LIBS:Microchip Technologies
 LIBS:analog_switches
 LIBS:motorola
-LIBS:texas
+LIBS:TI
 LIBS:intel
 LIBS:audio
@@
 LIBS:stepstick
 LIBS:Linear Technologies
-LIBS:Microchip Technologies
 LIBS:Maxim Integrated
 LIBS:Intersil
 LIBS:mounting hole
-LIBS:TI
 LIBS:power_transistors
 LIBS:FireMC-3.14-cache
@@
 $EndComp
 $Comp
-L MCP23S17 U3
-U 1 1 57D1D763
-P 8900 5200
-F 0 "U3" H 9150 6150 50  0000 R CNN
-F 1 "MCP23S17" H 8900 4250 50  0000 C CNN
-F 2 "IPC_SOIC127P:SOIC127P1030X265-28N" H 8450 4550 50  0001 C CNN
-F 3 "" H 8450 4550 50  0000 C CNN
-	1    8900 5200
-	1    0    0    -1
-$EndComp
-$Comp
 L VCC #PWR028
 U 1 1 57D1D96E
@@
 Wire Wire Line
 	2400 1800 3000 1800
+$Comp
+L MCP23S17 U?
+U 1 1 58B3320A
+P 8900 5200
+F 0 "U?" H 9150 6150 50  0000 R CNN
+F 1 "MCP23S17" H 8900 4250 50  0000 C CNN
+F 2 "" H 8450 4550 50  0000 C CNN
+F 3 "" H 8450 4550 50  0000 C CNN
+	1    8900 5200
+	1    0    0    -1
+$EndComp
 $EndSCHEMATC

Commit message: update
Parts:
- U3: renamed from U?; footprint (none) -> IPC_SOIC127P:SOIC127P1030X265-28N
Connections:
- net GPIO24: no longer names the net of J4.18
- net GPIO25: no longer names the net of J4.22
- net GPIO25: no longer J4.37
- net GPIO27: no longer names the net of J4.13
- net GPIO5: no longer names the net of J4.29
- net GPIO6: no longer names the net of J4.31
- net ID_SC: no longer names the net of J4.28
- net ID_SD: no longer names the net of J4.27
- net SCL1: no longer names the net of J4.5
- net SDA1: no longer names the net of J4.3
- net SPI_CE1: no longer names the net of J4.26
- no-connect marks 17 -> 28
Changed lines of the file:
@@
 	3700 1900 3800 1900
 Wire Wire Line
-	3800 1900 3800 3700
-Wire Wire Line
-	3700 3300 3800 3300
+	3800 3300 3700 3300
 Connection ~ 3800 3300
 Wire Wire Line
-	3700 3100 3800 3100
+	3800 3100 3700 3100
 Connection ~ 3800 3100
 Wire Wire Line
-	3700 2600 3800 2600
+	3800 2600 3700 2600
 Connection ~ 3800 2600
 Wire Wire Line
@@
 	3000 2100 2900 2100
 Wire Wire Line
-	2900 2100 2900 3700
-Wire Wire Line
-	3000 3600 2900 3600
+	2900 3600 3000 3600
 Connection ~ 2900 3600
 Wire Wire Line
@@
 	2400 2800 3000 2800
 Wire Wire Line
-	2400 1900 3000 1900
-Wire Wire Line
-	3700 2900 4300 2900
-Wire Wire Line
 	3700 2800 4300 2800
 $Comp
-L GND #PWR015
-U 1 1 57CB4DBD
-P 2900 3700
-F 0 "#PWR015" H 2900 3450 50  0001 C CNN
-F 1 "GND" H 2900 3550 50  0000 C CNN
-F 2 "" H 2900 3700 50  0000 C CNN
-F 3 "" H 2900 3700 50  0000 C CNN
-	1    2900 3700
-	1    0    0    -1
-$EndComp
-$Comp
-L GND #PWR016
+L GND #PWR017
 U 1 1 57CB4DD3
 P 3800 3700
-F 0 "#PWR016" H 3800 3450 50  0001 C CNN
+F 0 "#PWR017" H 3800 3450 50  0001 C CNN
 F 1 "GND" H 3800 3550 50  0000 C CNN
 F 2 "" H 3800 3700 50  0000 C CNN
@@
 	3700 2400 4300 2400
 Wire Wire Line
-	3700 2500 4300 2500
-Wire Wire Line
-	2400 2000 3000 2000
-Wire Wire Line
-	2400 2200 3000 2200
-Wire Wire Line
-	2400 2300 3000 2300
-Wire Wire Line
-	2400 2400 3000 2400
-Wire Wire Line
-	2400 3100 3000 3100
-Wire Wire Line
-	2400 3200 3000 3200
-Wire Wire Line
 	2400 3300 3000 3300
 Wire Wire Line
 	2400 3400 3000 3400
 Wire Wire Line
-	2400 3500 3000 3500
-Wire Wire Line
 	3700 3600 4300 3600
 Wire Wire Line
@@
 Wire Wire Line
 	3700 3200 4300 3200
-Wire Wire Line
-	3700 2700 4300 2700
 $Comp
 L Header_1X4 J3
@@
 $EndComp
 $Comp
-L GND #PWR017
+L GND #PWR018
 U 1 1 57CB72B4
 P 8400 2100
-F 0 "#PWR017" H 8400 1850 50  0001 C CNN
+F 0 "#PWR018" H 8400 1850 50  0001 C CNN
 F 1 "GND" H 8400 1950 50  0000 C CNN
 F 2 "" H 8400 2100 50  0000 C CNN
@@
 $EndComp
 $Comp
-L +5V #PWR018
+L +5V #PWR019
 U 1 1 57CB7418
 P 8400 1600
-F 0 "#PWR018" H 8400 1450 50  0001 C CNN
+F 0 "#PWR019" H 8400 1450 50  0001 C CNN
 F 1 "+5V" H 8400 1740 50  0000 C CNN
 F 2 "" H 8400 1600 50  0000 C CNN
@@
 NoConn ~ 8500 1800
 NoConn ~ 8500 1900
-Text GLabel 2400 1800 0    50   Input ~ 0
-SDA1
-Text GLabel 2400 1900 0    50   Input ~ 0
-SCL1
 Text GLabel 2400 2000 0    50   Input ~ 0
 ~ALLSTOP
 Text GLabel 2400 2200 0    50   Input ~ 0
 STEP2
-Text GLabel 2400 2300 0    50   Input ~ 0
-GPIO27
 Text GLabel 2400 2400 0    50   Input ~ 0
 ZMAX
@@
 Text GLabel 7600 5100 0    50   Input ~ 0
 SPI_SLCK
-Text GLabel 2400 3000 0    50   Input ~ 0
-ID_SD
-Text GLabel 2400 3100 0    50   Input ~ 0
-GPIO5
-Text GLabel 2400 3200 0    50   Input ~ 0
-GPIO6
 Text GLabel 2400 3300 0    50   Input ~ 0
 DIR2
 Text GLabel 2400 3400 0    50   Input ~ 0
 STEP4
-Text GLabel 2400 3500 0    50   Input ~ 0
-GPIO25
 Text GLabel 4300 2000 2    50   Input ~ 0
 DIR3
@@
 Text GLabel 4300 2400 2    50   Input ~ 0
 EMAX
-Text GLabel 4300 2500 2    50   Input ~ 0
-GPIO24
-Text GLabel 4300 2700 2    50   Input ~ 0
-GPIO25
 Text GLabel 4300 2800 2    50   Input ~ 0
 SPI_CE0
-Text GLabel 4300 2900 2    50   Input ~ 0
-SPI_CE1
-Text GLabel 4300 3000 2    50   Input ~ 0
-ID_SC
 Text GLabel 4300 3200 2    50   Input ~ 0
 DIR1
@@
 $EndComp
 $Comp
-L VCC #PWR019
+L VCC #PWR020
 U 1 1 57D1D60D
 P 1300 7250
-F 0 "#PWR019" H 1300 7100 50  0001 C CNN
+F 0 "#PWR020" H 1300 7100 50  0001 C CNN
 F 1 "VCC" H 1300 7400 50  0000 C CNN
 F 2 "" H 1300 7250 50  0000 C CNN
@@
 $EndComp
 $Comp
-L VCC #PWR020
+L VCC #PWR021
 U 1 1 57D1D63A
 P 3500 7250
-F 0 "#PWR020" H 3500 7100 50  0001 C CNN
+F 0 "#PWR021" H 3500 7100 50  0001 C CNN
 F 1 "VCC" H 3500 7400 50  0000 C CNN
 F 2 "" H 3500 7250 50  0000 C CNN
@@
 $EndComp
 $Comp
-L VCC #PWR021
+L VCC #PWR022
 U 1 1 57D1D660
 P 4900 4700
-F 0 "#PWR021" H 4900 4550 50  0001 C CNN
+F 0 "#PWR022" H 4900 4550 50  0001 C CNN
 F 1 "VCC" H 4900 4850 50  0000 C CNN
 F 2 "" H 4900 4700 50  0000 C CNN
@@
 $EndComp
 $Comp
-L VCC #PWR022
+L VCC #PWR023
 U 1 1 57D1D686
 P 4600 7250
-F 0 "#PWR022" H 4600 7100 50  0001 C CNN
+F 0 "#PWR023" H 4600 7100 50  0001 C CNN
 F 1 "VCC" H 4600 7400 50  0000 C CNN
 F 2 "" H 4600 7250 50  0000 C CNN
@@
 $EndComp
 $Comp
-L GND #PWR023
+L GND #PWR024
 U 1 1 57D1D6AC
 P 1300 7650
-F 0 "#PWR023" H 1300 7400 50  0001 C CNN
+F 0 "#PWR024" H 1300 7400 50  0001 C CNN
 F 1 "GND" H 1300 7500 50  0000 C CNN
 F 2 "" H 1300 7650 50  0000 C CNN
@@
 $EndComp
 $Comp
-L GND #PWR024
+L GND #PWR025
 U 1 1 57D1D6D2
 P 1600 5800
-F 0 "#PWR024" H 1600 5550 50  0001 C CNN
+F 0 "#PWR025" H 1600 5550 50  0001 C CNN
 F 1 "GND" H 1600 5650 50  0000 C CNN
 F 2 "" H 1600 5800 50  0000 C CNN
@@
 $EndComp
 $Comp
-L GND #PWR025
+L GND #PWR026
 U 1 1 57D1D6F8
 P 3200 5800
-F 0 "#PWR025" H 3200 5550 50  0001 C CNN
+F 0 "#PWR026" H 3200 5550 50  0001 C CNN
 F 1 "GND" H 3200 5650 50  0000 C CNN
 F 2 "" H 3200 5800 50  0000 C CNN
@@
 $EndComp
 $Comp
-L GND #PWR026
+L GND #PWR027
 U 1 1 57D1D71E
 P 4900 5800
-F 0 "#PWR026" H 4900 5550 50  0001 C CNN
+F 0 "#PWR027" H 4900 5550 50  0001 C CNN
 F 1 "GND" H 4900 5650 50  0000 C CNN
 F 2 "" H 4900 5800 50  0000 C CNN
@@
 $EndComp
 $Comp
-L GND #PWR027
+L GND #PWR028
 U 1 1 57D1D744
 P 4600 7650
-F 0 "#PWR027" H 4600 7400 50  0001 C CNN
+F 0 "#PWR028" H 4600 7400 50  0001 C CNN
 F 1 "GND" H 4600 7500 50  0000 C CNN
 F 2 "" H 4600 7650 50  0000 C CNN
@@
 $EndComp
 $Comp
-L VCC #PWR028
+L VCC #PWR029
 U 1 1 57D1D96E
 P 7700 4300
-F 0 "#PWR028" H 7700 4150 50  0001 C CNN
+F 0 "#PWR029" H 7700 4150 50  0001 C CNN
 F 1 "VCC" H 7700 4450 50  0000 C CNN
 F 2 "" H 7700 4300 50  0000 C CNN
@@
 $EndComp
 $Comp
-L GND #PWR029
+L GND #PWR030
 U 1 1 57D1D997
 P 8300 6100
-F 0 "#PWR029" H 8300 5850 50  0001 C CNN
+F 0 "#PWR030" H 8300 5850 50  0001 C CNN
 F 1 "GND" H 8300 5950 50  0000 C CNN
 F 2 "" H 8300 6100 50  0000 C CNN
@@
 	1300 7350 1300 7250
 $Comp
-L VCC #PWR030
+L VCC #PWR031
 U 1 1 57D1DEB5
 P 2400 7250
-F 0 "#PWR030" H 2400 7100 50  0001 C CNN
+F 0 "#PWR031" H 2400 7100 50  0001 C CNN
 F 1 "VCC" H 2400 7400 50  0000 C CNN
 F 2 "" H 2400 7250 50  0000 C CNN
@@
 $EndComp
 $Comp
-L VCC #PWR031
+L VCC #PWR032
 U 1 1 57D1DEDE
 P 3200 4700
-F 0 "#PWR031" H 3200 4550 50  0001 C CNN
+F 0 "#PWR032" H 3200 4550 50  0001 C CNN
 F 1 "VCC" H 3200 4850 50  0000 C CNN
 F 2 "" H 3200 4700 50  0000 C CNN
@@
 $EndComp
 $Comp
-L VCC #PWR032
+L VCC #PWR033
 U 1 1 57D1DF07
 P 1600 4700
-F 0 "#PWR032" H 1600 4550 50  0001 C CNN
+F 0 "#PWR033" H 1600 4550 50  0001 C CNN
 F 1 "VCC" H 1600 4850 50  0000 C CNN
 F 2 "" H 1600 4700 50  0000 C CNN
@@
 $EndComp
 $Comp
-L GND #PWR033
+L GND #PWR034
 U 1 1 57D1DF30
 P 3500 7650
-F 0 "#PWR033" H 3500 7400 50  0001 C CNN
+F 0 "#PWR034" H 3500 7400 50  0001 C CNN
 F 1 "GND" H 3500 7500 50  0000 C CNN
 F 2 "" H 3500 7650 50  0000 C CNN
@@
 $EndComp
 $Comp
-L GND #PWR034
+L GND #PWR035
 U 1 1 57D1DF59
 P 2400 7650
-F 0 "#PWR034" H 2400 7400 50  0001 C CNN
+F 0 "#PWR035" H 2400 7400 50  0001 C CNN
 F 1 "GND" H 2400 7500 50  0000 C CNN
 F 2 "" H 2400 7650 50  0000 C CNN
@@
 NoConn ~ 8400 5700
 NoConn ~ 8400 5800
-Wire Wire Line
-	2400 3000 3000 3000
-Wire Wire Line
-	3700 3000 4300 3000
-Wire Wire Line
-	2400 1800 3000 1800
-$Comp
-L MCP23S17 U?
+$Comp
+L MCP23S17 U3
 U 1 1 58B3320A
 P 8900 5200
-F 0 "U?" H 9150 6150 50  0000 R CNN
+F 0 "U3" H 9150 6150 50  0000 R CNN
 F 1 "MCP23S17" H 8900 4250 50  0000 C CNN
-F 2 "" H 8450 4550 50  0000 C CNN
+F 2 "IPC_SOIC127P:SOIC127P1030X265-28N" H 8450 4550 50  0001 C CNN
 F 3 "" H 8450 4550 50  0000 C CNN
 	1    8900 5200
 	1    0    0    -1
 $EndComp
+Wire Wire Line
+	3000 2000 2400 2000
+Wire Wire Line
+	3000 2200 2400 2200
+Wire Wire Line
+	3000 2400 2400 2400
+Wire Wire Line
+	2900 2100 2900 3700
+NoConn ~ 3000 3000
+NoConn ~ 3700 3000
+NoConn ~ 3000 3500
+NoConn ~ 3000 3100
+NoConn ~ 3700 2700
+NoConn ~ 3700 2500
+NoConn ~ 3000 2300
+NoConn ~ 3000 1900
+NoConn ~ 3000 1800
+$Comp
+L GND #PWR036
+U 1 1 591E7AD0
+P 2900 3700
+F 0 "#PWR036" H 2900 3450 50  0001 C CNN
+F 1 "GND" H 2900 3550 50  0000 C CNN
+F 2 "" H 2900 3700 50  0001 C CNN
+F 3 "" H 2900 3700 50  0001 C CNN
+	1    2900 3700
+	1    0    0    -1
+$EndComp
+NoConn ~ 3000 3200
+NoConn ~ 3700 2900
+Wire Wire Line
+	3800 1900 3800 3700
 $EndSCHEMATC
