File: FireMC-3.14.sch (KiCad schematic (older format))
At the start: 0 parts

Commit message: PCB Layout experimentation
Changed lines of the file:
@@
 $Descr A 11000 8500
 encoding utf-8
-Sheet 1 4
+Sheet 1 5
 Title "FireMC-3.14"
 Date ""
@@
 F1 "FireMC-3.14_PWR.sch" 60
 $EndSheet
+$Sheet
+S 9050 5300 1100 150
+U 57E0F559
+F0 "Safety" 50
+F1 "FireMC-3.14_SFTY.sch" 50
+$EndSheet
 $EndSCHEMATC

Commit message: Time to Update.  Board layout started.
Changed lines of the file:
@@
 LIBS:Maxim Integrated
 LIBS:Intersil
+LIBS:mounting hole
 LIBS:FireMC-3.14-cache
 EELAYER 25 0
@@
 $Sheet
 S 9050 6500 1100 150
-U 57C93439
-F0 "Motors" 60
-F1 "FireMC-3.14_MTR.sch" 60
+U 57C8E291
+F0 "Power" 60
+F1 "FireMC-3.14_PWR.sch" 60
 $EndSheet
 $Sheet
@@
 $Sheet
 S 9050 5700 1100 150
-U 57C8E291
-F0 "Power" 60
-F1 "FireMC-3.14_PWR.sch" 60
+U 57C93439
+F0 "Motors" 60
+F1 "FireMC-3.14_MTR.sch" 60
 $EndSheet
 $Sheet
