File: FireMC-3.14_MTR.sch (KiCad schematic (older format))
At the start: 28 parts, among them J10 Header_2X3, J11 Header_2X3, J3 Header_1X4, J4 Header_1X4, J6 Header_2X3, J7 Header_2X3, J8 Header_1X4, J9 Header_1X4, U3 TMC_SILENT_STEPSTICK, U4 TMC_SILENT_STEPSTICK, U7 TMC_SILENT_STEPSTICK, U8 TMC_SILENT_STEPSTICK

Commit message: Time to Update.  Board layout started.
Parts:
- added MH1, MH2, MH3, MH4: MOUNT_PTH, IPC_MFG:IMELLC_PTH_2.75x6.00, symbol MOUNT_PTH
- renumbered U7 to U5, U8 to U6
Connections:
- net GND: now also MH1.1, MH2.1, MH3.1, MH4.1
Changed lines of the file:
@@
 LIBS:Maxim Integrated
 LIBS:Intersil
+LIBS:mounting hole
 LIBS:FireMC-3.14-cache
 EELAYER 25 0
@@
 $Descr A 11000 8500
 encoding utf-8
-Sheet 2 5
+Sheet 4 5
 Title "FireMC-3.14"
 Date ""
@@
 $EndComp
 $Comp
-L TMC_SILENT_STEPSTICK U7
+L TMC_SILENT_STEPSTICK U5
 U 1 1 57CC8D2D
 P 7800 1650
-F 0 "U7" H 8100 2100 60  0000 R BNN
+F 0 "U5" H 8100 2100 60  0000 R BNN
 F 1 "TMC_SILENT_STEPSTICK" H 7800 1200 60  0000 C CNN
 F 2 "IPC_MFG:stepstick" H 7800 1650 60  0001 C CNN
@@
 $EndComp
 $Comp
-L TMC_SILENT_STEPSTICK U8
+L TMC_SILENT_STEPSTICK U6
 U 1 1 57CC8D78
 P 7800 4100
-F 0 "U8" H 8100 4550 60  0000 R BNN
+F 0 "U6" H 8100 4550 60  0000 R BNN
 F 1 "TMC_SILENT_STEPSTICK" H 7800 3650 60  0000 C CNN
 F 2 "IPC_MFG:stepstick" H 7800 4100 60  0001 C CNN
@@
 $EndComp
 $Comp
-L GND #PWR01
+L GND #PWR028
 U 1 1 57CC93BA
 P 1800 2700
-F 0 "#PWR01" H 1800 2450 50  0001 C CNN
+F 0 "#PWR028" H 1800 2450 50  0001 C CNN
 F 1 "GND" H 1800 2550 50  0000 C CNN
 F 2 "" H 1800 2700 50  0000 C CNN
@@
 $EndComp
 $Comp
-L GND #PWR02
+L GND #PWR029
 U 1 1 57CC93F0
 P 1800 5150
-F 0 "#PWR02" H 1800 4900 50  0001 C CNN
+F 0 "#PWR029" H 1800 4900 50  0001 C CNN
 F 1 "GND" H 1800 5000 50  0000 C CNN
 F 2 "" H 1800 5150 50  0000 C CNN
@@
 $EndComp
 $Comp
-L GND #PWR03
+L GND #PWR030
 U 1 1 57CC94AF
 P 7100 2700
-F 0 "#PWR03" H 7100 2450 50  0001 C CNN
+F 0 "#PWR030" H 7100 2450 50  0001 C CNN
 F 1 "GND" H 7100 2550 50  0000 C CNN
 F 2 "" H 7100 2700 50  0000 C CNN
@@
 $EndComp
 $Comp
-L GND #PWR04
+L GND #PWR031
 U 1 1 57CC94DE
 P 7100 5150
-F 0 "#PWR04" H 7100 4900 50  0001 C CNN
+F 0 "#PWR031" H 7100 4900 50  0001 C CNN
 F 1 "GND" H 7100 5000 50  0000 C CNN
 F 2 "" H 7100 5150 50  0000 C CNN
@@
 	3300 2500 3300 2700
 $Comp
-L GND #PWR05
+L GND #PWR032
 U 1 1 57CCD112
 P 3300 2700
-F 0 "#PWR05" H 3300 2450 50  0001 C CNN
+F 0 "#PWR032" H 3300 2450 50  0001 C CNN
 F 1 "GND" H 3300 2550 50  0000 C CNN
 F 2 "" H 3300 2700 50  0000 C CNN
@@
 DIR2
 $Comp
-L GND #PWR06
+L GND #PWR033
 U 1 1 57CCD523
 P 3300 5150
-F 0 "#PWR06" H 3300 4900 50  0001 C CNN
+F 0 "#PWR033" H 3300 4900 50  0001 C CNN
 F 1 "GND" H 3300 5000 50  0000 C CNN
 F 2 "" H 3300 5150 50  0000 C CNN
@@
 	8700 1200 9000 1200
 $Comp
-L GND #PWR07
+L GND #PWR034
 U 1 1 57CD09E3
 P 8600 2700
-F 0 "#PWR07" H 8600 2450 50  0001 C CNN
+F 0 "#PWR034" H 8600 2450 50  0001 C CNN
 F 1 "GND" H 8600 2550 50  0000 C CNN
 F 2 "" H 8600 2700 50  0000 C CNN
@@
 	8700 4150 8900 4150
 $Comp
-L GND #PWR08
+L GND #PWR035
 U 1 1 57CD40F0
 P 8600 5150
-F 0 "#PWR08" H 8600 4900 50  0001 C CNN
+F 0 "#PWR035" H 8600 4900 50  0001 C CNN
 F 1 "GND" H 8600 5000 50  0000 C CNN
 F 2 "" H 8600 5150 50  0000 C CNN
@@
 EN4_O
 $Comp
-L +12V #PWR09
+L +12V #PWR036
 U 1 1 57D19E3A
 P 1400 1200
-F 0 "#PWR09" H 1400 1050 50  0001 C CNN
+F 0 "#PWR036" H 1400 1050 50  0001 C CNN
 F 1 "+12V" H 1400 1340 50  0000 C CNN
 F 2 "" H 1400 1200 50  0000 C CNN
@@
 $EndComp
 $Comp
-L VCC #PWR010
+L VCC #PWR037
 U 1 1 57D19E76
 P 1600 1200
-F 0 "#PWR010" H 1600 1050 50  0001 C CNN
+F 0 "#PWR037" H 1600 1050 50  0001 C CNN
 F 1 "VCC" H 1600 1350 50  0000 C CNN
 F 2 "" H 1600 1200 50  0000 C CNN
@@
 $EndComp
 $Comp
-L +12V #PWR011
+L +12V #PWR038
 U 1 1 57D19EC4
 P 1400 3650
-F 0 "#PWR011" H 1400 3500 50  0001 C CNN
+F 0 "#PWR038" H 1400 3500 50  0001 C CNN
 F 1 "+12V" H 1400 3790 50  0000 C CNN
 F 2 "" H 1400 3650 50  0000 C CNN
@@
 $EndComp
 $Comp
-L +12V #PWR012
+L +12V #PWR039
 U 1 1 57D19F0B
 P 6700 3650
-F 0 "#PWR012" H 6700 3500 50  0001 C CNN
+F 0 "#PWR039" H 6700 3500 50  0001 C CNN
 F 1 "+12V" H 6700 3790 50  0000 C CNN
 F 2 "" H 6700 3650 50  0000 C CNN
@@
 $EndComp
 $Comp
-L +12V #PWR013
+L +12V #PWR040
 U 1 1 57D19F52
 P 6700 1200
-F 0 "#PWR013" H 6700 1050 50  0001 C CNN
+F 0 "#PWR040" H 6700 1050 50  0001 C CNN
 F 1 "+12V" H 6700 1340 50  0000 C CNN
 F 2 "" H 6700 1200 50  0000 C CNN
@@
 $EndComp
 $Comp
-L VCC #PWR014
+L VCC #PWR041
 U 1 1 57D19F99
 P 1600 3650
-F 0 "#PWR014" H 1600 3500 50  0001 C CNN
+F 0 "#PWR041" H 1600 3500 50  0001 C CNN
 F 1 "VCC" H 1600 3800 50  0000 C CNN
 F 2 "" H 1600 3650 50  0000 C CNN
@@
 $EndComp
 $Comp
-L VCC #PWR015
+L VCC #PWR042
 U 1 1 57D19FE0
 P 4500 1500
-F 0 "#PWR015" H 4500 1350 50  0001 C CNN
+F 0 "#PWR042" H 4500 1350 50  0001 C CNN
 F 1 "VCC" H 4500 1650 50  0000 C CNN
 F 2 "" H 4500 1500 50  0000 C CNN
@@
 $EndComp
 $Comp
-L VCC #PWR016
+L VCC #PWR043
 U 1 1 57D1A03C
 P 4500 3950
-F 0 "#PWR016" H 4500 3800 50  0001 C CNN
+F 0 "#PWR043" H 4500 3800 50  0001 C CNN
 F 1 "VCC" H 4500 4100 50  0000 C CNN
 F 2 "" H 4500 3950 50  0000 C CNN
@@
 $EndComp
 $Comp
-L VCC #PWR017
+L VCC #PWR044
 U 1 1 57D1A083
 P 6900 3650
-F 0 "#PWR017" H 6900 3500 50  0001 C CNN
+F 0 "#PWR044" H 6900 3500 50  0001 C CNN
 F 1 "VCC" H 6900 3800 50  0000 C CNN
 F 2 "" H 6900 3650 50  0000 C CNN
@@
 $EndComp
 $Comp
-L VCC #PWR018
+L VCC #PWR045
 U 1 1 57D1A0CA
 P 9800 3950
-F 0 "#PWR018" H 9800 3800 50  0001 C CNN
+F 0 "#PWR045" H 9800 3800 50  0001 C CNN
 F 1 "VCC" H 9800 4100 50  0000 C CNN
 F 2 "" H 9800 3950 50  0000 C CNN
@@
 $EndComp
 $Comp
-L VCC #PWR019
+L VCC #PWR046
 U 1 1 57D1A111
 P 9800 1500
-F 0 "#PWR019" H 9800 1350 50  0001 C CNN
+F 0 "#PWR046" H 9800 1350 50  0001 C CNN
 F 1 "VCC" H 9800 1650 50  0000 C CNN
 F 2 "" H 9800 1500 50  0000 C CNN
@@
 $EndComp
 $Comp
-L VCC #PWR020
+L VCC #PWR047
 U 1 1 57D1A158
 P 6900 1200
-F 0 "#PWR020" H 6900 1050 50  0001 C CNN
+F 0 "#PWR047" H 6900 1050 50  0001 C CNN
 F 1 "VCC" H 6900 1350 50  0000 C CNN
 F 2 "" H 6900 1200 50  0000 C CNN
@@
 Connection ~ 3200 4450
 $Comp
-L VCC #PWR021
+L VCC #PWR048
 U 1 1 57D5AA58
 P 3200 3250
-F 0 "#PWR021" H 3200 3100 50  0001 C CNN
+F 0 "#PWR048" H 3200 3100 50  0001 C CNN
 F 1 "VCC" H 3200 3400 50  0000 C CNN
 F 2 "" H 3200 3250 50  0000 C CNN
@@
 $EndComp
 $Comp
-L VCC #PWR022
+L VCC #PWR049
 U 1 1 57D5B02E
 P 3200 800
-F 0 "#PWR022" H 3200 650 50  0001 C CNN
+F 0 "#PWR049" H 3200 650 50  0001 C CNN
 F 1 "VCC" H 3200 950 50  0000 C CNN
 F 2 "" H 3200 800 50  0000 C CNN
@@
 $EndComp
 $Comp
-L VCC #PWR023
+L VCC #PWR050
 U 1 1 57D5B08D
 P 8500 800
-F 0 "#PWR023" H 8500 650 50  0001 C CNN
+F 0 "#PWR050" H 8500 650 50  0001 C CNN
 F 1 "VCC" H 8500 950 50  0000 C CNN
 F 2 "" H 8500 800 50  0000 C CNN
@@
 $EndComp
 $Comp
-L VCC #PWR024
+L VCC #PWR051
 U 1 1 57D5B0EC
 P 8500 3250
-F 0 "#PWR024" H 8500 3100 50  0001 C CNN
+F 0 "#PWR051" H 8500 3100 50  0001 C CNN
 F 1 "VCC" H 8500 3400 50  0000 C CNN
 F 2 "" H 8500 3250 50  0000 C CNN
@@
 Wire Wire Line
 	3100 4050 3000 4050
+$Comp
+L MOUNT_PTH MH1
+U 1 1 57E613F9
+P 1700 5850
+F 0 "MH1" H 1700 5950 50  0000 C CNN
+F 1 "MOUNT_PTH" H 1700 5750 50  0000 C CNN
+F 2 "IPC_MFG:IMELLC_PTH_2.75x6.00" H 1700 5850 50  0001 C CNN
+F 3 "" H 1700 5850 50  0000 C CNN
+	1    1700 5850
+	1    0    0    -1
+$EndComp
+$Comp
+L MOUNT_PTH MH2
+U 1 1 57E6149B
+P 1700 6150
+F 0 "MH2" H 1700 6250 50  0000 C CNN
+F 1 "MOUNT_PTH" H 1700 6050 50  0000 C CNN
+F 2 "IPC_MFG:IMELLC_PTH_2.75x6.00" H 1700 6150 50  0001 C CNN
+F 3 "" H 1700 6150 50  0000 C CNN
+	1    1700 6150
+	1    0    0    -1
+$EndComp
+$Comp
+L MOUNT_PTH MH3
+U 1 1 57E6150D
+P 1700 6450
+F 0 "MH3" H 1700 6550 50  0000 C CNN
+F 1 "MOUNT_PTH" H 1700 6350 50  0000 C CNN
+F 2 "IPC_MFG:IMELLC_PTH_2.75x6.00" H 1700 6450 50  0001 C CNN
+F 3 "" H 1700 6450 50  0000 C CNN
+	1    1700 6450
+	1    0    0    -1
+$EndComp
+$Comp
+L MOUNT_PTH MH4
+U 1 1 57E61582
+P 1700 6750
+F 0 "MH4" H 1700 6850 50  0000 C CNN
+F 1 "MOUNT_PTH" H 1700 6650 50  0000 C CNN
+F 2 "IPC_MFG:IMELLC_PTH_2.75x6.00" H 1700 6750 50  0001 C CNN
+F 3 "" H 1700 6750 50  0000 C CNN
+	1    1700 6750
+	1    0    0    -1
+$EndComp
+$Comp
+L GND #PWR052
+U 1 1 57E615DC
+P 1450 6850
+F 0 "#PWR052" H 1450 6600 50  0001 C CNN
+F 1 "GND" H 1450 6700 50  0000 C CNN
+F 2 "" H 1450 6850 50  0000 C CNN
+F 3 "" H 1450 6850 50  0000 C CNN
+	1    1450 6850
+	1    0    0    -1
+$EndComp
+Wire Wire Line
+	1450 5850 1450 6850
+Wire Wire Line
+	1450 6750 1550 6750
+Wire Wire Line
+	1450 6450 1550 6450
+Connection ~ 1450 6750
+Wire Wire Line
+	1450 6150 1550 6150
+Connection ~ 1450 6450
+Wire Wire Line
+	1450 5850 1550 5850
+Connection ~ 1450 6150
 $EndSCHEMATC

Commit message: Update 1/1/2017
Parts:
- removed MH1, MH2, MH3, MH4: MOUNT_PTH, IPC_MFG:IMELLC_PTH_2.75x6.00, symbol MOUNT_PTH
Changed lines of the file:
@@
 Wire Wire Line
 	3100 4050 3000 4050
-$Comp
-L MOUNT_PTH MH1
-U 1 1 57E613F9
-P 1700 5850
-F 0 "MH1" H 1700 5950 50  0000 C CNN
-F 1 "MOUNT_PTH" H 1700 5750 50  0000 C CNN
-F 2 "IPC_MFG:IMELLC_PTH_2.75x6.00" H 1700 5850 50  0001 C CNN
-F 3 "" H 1700 5850 50  0000 C CNN
-	1    1700 5850
-	1    0    0    -1
-$EndComp
-$Comp
-L MOUNT_PTH MH2
-U 1 1 57E6149B
-P 1700 6150
-F 0 "MH2" H 1700 6250 50  0000 C CNN
-F 1 "MOUNT_PTH" H 1700 6050 50  0000 C CNN
-F 2 "IPC_MFG:IMELLC_PTH_2.75x6.00" H 1700 6150 50  0001 C CNN
-F 3 "" H 1700 6150 50  0000 C CNN
-	1    1700 6150
-	1    0    0    -1
-$EndComp
-$Comp
-L MOUNT_PTH MH3
-U 1 1 57E6150D
-P 1700 6450
-F 0 "MH3" H 1700 6550 50  0000 C CNN
-F 1 "MOUNT_PTH" H 1700 6350 50  0000 C CNN
-F 2 "IPC_MFG:IMELLC_PTH_2.75x6.00" H 1700 6450 50  0001 C CNN
-F 3 "" H 1700 6450 50  0000 C CNN
-	1    1700 6450
-	1    0    0    -1
-$EndComp
-$Comp
-L MOUNT_PTH MH4
-U 1 1 57E61582
-P 1700 6750
-F 0 "MH4" H 1700 6850 50  0000 C CNN
-F 1 "MOUNT_PTH" H 1700 6650 50  0000 C CNN
-F 2 "IPC_MFG:IMELLC_PTH_2.75x6.00" H 1700 6750 50  0001 C CNN
-F 3 "" H 1700 6750 50  0000 C CNN
-	1    1700 6750
-	1    0    0    -1
-$EndComp
-$Comp
-L GND #PWR052
-U 1 1 57E615DC
-P 1450 6850
-F 0 "#PWR052" H 1450 6600 50  0001 C CNN
-F 1 "GND" H 1450 6700 50  0000 C CNN
-F 2 "" H 1450 6850 50  0000 C CNN
-F 3 "" H 1450 6850 50  0000 C CNN
-	1    1450 6850
-	1    0    0    -1
-$EndComp
-Wire Wire Line
-	1450 5850 1450 6850
-Wire Wire Line
-	1450 6750 1550 6750
-Wire Wire Line
-	1450 6450 1550 6450
-Connection ~ 1450 6750
-Wire Wire Line
-	1450 6150 1550 6150
-Connection ~ 1450 6450
-Wire Wire Line
-	1450 5850 1550 5850
-Connection ~ 1450 6150
 $EndSCHEMATC

Commit message: Changed Power management
Parts:
- renumbered C37 to C21, C40 to C22, C38 to C23, C41 to C24, J3 to J12, J8 to J13, J6 to J14, J10 to J15, J4 to J16, J9 to J17, J7 to J18, J11 to J19, R17 to R18, R23 to R19, R19 to R20, R25 to R22, R27 to R23, R18 to R24, R24 to R25, R20 to R26, R22 to R27, R26 to R28, R28 to R29, U3 to U4, U4 to U6, U6 to U7
