File: FireMC-3.14_PWR.sch (KiCad schematic (older format))
At the start: 28 parts, among them J1 Header_1X4, Q1 STD86N3LH5, Q2 STD86N3LH5, U1 ISL6420B

Commit message: Schematic Update and Design Calcs for 3V3
Parts:
- added C13: 6n8, symbol C
- added R1: 10k, symbol R
- added R2: 1k, symbol R
- added R7: 158R, symbol R
- C10: value C -> 156n
- C11: value C -> 560p
- C12: value C -> 1n6
- C7: value C -> 10n
- C9: value C -> 0u1
- L1: value 8u2 -> 6u8
- R3: renamed from R1; value R -> 5k76
- R4: renamed from R2; value R -> 56k2
- R5: renamed from R4; value R -> 2k21
- R6: renamed from R3; value R -> 10k
- gave numbers to parts that had none: 3
- renumbered C13 to C14
Connections:
- wire segments 86 -> 93
Other:
- moved on the sheet: C10, C11, C12, C14, C15, C16, C2, C3, C4, C5, C6, C7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

Commit message: math check
Parts:
- removed F1: 3A, symbol FUSE
- removed F2: 10A, symbol FUSE
- removed F3: 5A, symbol FUSE
- removed J1: Header_1X4, symbol Header_1X4
- added C18, C19: 10u, symbol C
- added C20, C21: 4u7, symbol C
- added C22, C25, C26: 0u1, symbol C
- added C23: 2u2, symbol C
- added C24: 10n, symbol C
- added C27: 156n, symbol C
- added C28: 560p, symbol C
- added C29: 1n6, symbol C
- added C30: 6n8, symbol C
- added C31, C32, C33: 150u, symbol CP1
- added D2: PMEG3050EP,115, symbol D_Schottky
- added F1: 10A, symbol F_Small
- added F2, F3: 4A, symbol F_Small
- added J1, J2: Header_1X2, symbol Header_1X2
- added L?: 6u8, symbol INDUCTOR
- added Q3, Q4: STD86N3LH5, symbol Q_NMOS_GDS
- added R10: 5k76, symbol R
- added R11: 56k2, symbol R
- added R12: 2k21, symbol R
- added R13, R8: 10k, symbol R
- added R14: 158R, symbol R
- added R9: 1k, symbol R
- added U2: ISL6420B, symbol ISL6420B
- R2: value 1k -> 2k5
Connections:
- net labels added: VCC
- net labels removed: +12LF, +5C, +5F
- wire segments 93 -> 173
Other:
- moved on the sheet: C1, C10, C11, C12, C13, C14, C15, C16, C2, C3, C4, C5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

Commit message: Schematic 80% complete
Parts:
- added C22, C23, C4, C5: 10u, symbol C
- added D? (x3): LED, symbol LED
- added R? (x3): 178R, symbol R
- C13: renamed from C11; value 560p -> 62p
- C14: renamed from C12; value 1n6 -> 1n3
- C15: renamed from C13; value 6n8 -> 5n6
- C21: renamed from C20; value 4u7 -> 10u
- C3: value 4u7 -> 10u
- C31: renamed from C28; value 560p -> 62p
- C32: renamed from C29; value 1n6 -> 1n5
- C33: renamed from C30; value 6n8 -> 6n2
- L2: renamed from L?; value 6u8 -> 8u2
- R10: value 5k76 -> 510R
- R12: value 2k21 -> 1k37
- R14: value 158R -> 178R
- R3: value 5k76 -> 499R
- R7: value 158R -> 196R
- renumbered C8 to C10, C9 to C11, C10 to C12, C14 to C16, C15 to C17, C16 to C18, C18 to C19, C19 to C20, C21 to C24, C22 to C25, C23 to C26, C24 to C27, C25 to C28, C26 to C29, C27 to C30, C31 to C34, C32 to C35, C33 to C36, C4 to C6, C5 to C7, C6 to C8, C7 to C9
Connections:
- net labels added: PGD3, PGD5
- wire segments 173 -> 194
Other:
- moved on the sheet: C10, C11, C12, C13, C14, C15, C16, C17, C18, C24, C25, C26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

Commit message: PCB Layout experimentation
Parts:
- C1, C19, C2, C20, C21, C22, C23, C24, C3, C4, C5, C6: footprint (none) -> IPC_CAP:CAPC1608X95N
- C10, C11, C13, C14, C15, C25, C26, C27, C28, C29, C31, C32, C33, C7, C8, C9: footprint (none) -> IPC_CAP:CAPC1608X90N
- C12: value 156n -> 180n; footprint (none) -> IPC_CAP:CAPC1608X90N
- C16, C17, C18, C34, C35, C36: footprint (none) -> IPC_CAP:CAPAE660X770N
- C30: value 156n -> 220n; footprint (none) -> IPC_CAP:CAPC1608X90N
- D1, D2: footprint (none) -> IPC_SOD:SOD4725X100N
- D3, D4, D5: renamed from D?; footprint (none) -> IPC_LED:LEDM1608X70N
- F1: footprint (none) -> IPC_MFG:MPD_BK-6010; Mfg PN (none) -> 0ATO010.V
- F2, F3: value 4A -> 5A; footprint (none) -> IPC_MFG:MPD_BK-6010; Mfg PN (none) -> 0ATO005.V
- J1: footprint (none) -> IPC_MFG:MOLEX_395321002
- J2: footprint (none) -> IPC_MFG:PHEONIX_1923869
- L1, L2: footprint (none) -> IPC_IND:INDM1213X620N
- Q1, Q2, Q3, Q4: footprint (none) -> IPC_TO:TO228P972X240-3N
- R1, R10, R11, R12, R13, R14, R2, R3, R4, R5, R6, R7, R8, R9: footprint (none) -> IPC_RES:RESC1608X55N
- R34, R35, R36: renamed from R?; value 178R -> 2k21; footprint (none) -> IPC_RES:RESC1608X55N
- U1, U2: footprint (none) -> IPC_SOP:SOP63P600X155-20N

Commit message: Time to Update.  Board layout started.
Parts:
- F1, F2, F3: symbol F_Small -> FUSE
Connections:
- net labels added: 12VIN, 3V3OUT, 5VOUT
Changed lines of the file:
@@
 LIBS:Maxim Integrated
 LIBS:Intersil
+LIBS:mounting hole
 LIBS:FireMC-3.14-cache
 EELAYER 25 0
@@
 $Descr A 11000 8500
 encoding utf-8
-Sheet 4 5
+Sheet 2 5
 Title "FireMC-3.14"
 Date ""
@@
 	4500 2700 4500 3000
 Wire Wire Line
-	4800 2500 3900 2500
+	3900 2500 4800 2500
 Wire Wire Line
 	4200 3000 4200 2500
@@
 Connection ~ 3300 1500
 Wire Wire Line
-	4800 1400 3000 1400
+	3000 1400 4800 1400
 Connection ~ 3000 1500
 Connection ~ 1500 1300
@@
 Connection ~ 1800 1300
 Wire Wire Line
-	2100 3000 2100 1300
+	2100 1300 2100 3000
 Connection ~ 2100 1300
 Wire Wire Line
-	1100 800  9800 800
+	1100 800  9750 800
 Wire Wire Line
 	3000 1000 5500 1000
@@
 Connection ~ 6700 1300
 Wire Wire Line
-	7650 1400 7650 800
+	7650 800  7650 1400
 Connection ~ 7650 800
 Connection ~ 7650 1900
@@
 Wire Wire Line
 	7100 3000 7100 2900
-Wire Wire Line
-	8500 1900 9800 1900
 Wire Wire Line
 	9000 2000 9000 1900
@@
 	8550 2500 8700 2500
 Wire Wire Line
-	8550 2800 8700 2800
-Wire Wire Line
-	8700 2800 8700 1900
+	8700 2800 8550 2800
+Wire Wire Line
+	8700 1900 8700 2800
 Connection ~ 9300 3500
 Connection ~ 9000 3500
@@
 Connection ~ 6800 3400
 Wire Wire Line
-	7450 3300 7450 3500
+	7450 3500 7450 3300
 Wire Wire Line
 	7100 3400 7100 3300
@@
 	9300 3500 9300 2300
 $Comp
-L F_Small F1
+L FUSE F1
 U 1 1 57D1191B
-P 9900 800
-F 0 "F1" H 9860 860 50  0000 L CNN
-F 1 "10A" H 9780 740 50  0000 L CNN
-F 2 "IPC_MFG:MPD_BK-6010" H 9900 800 50  0001 C CNN
-F 3 "" H 9900 800 50  0000 C CNN
-F 4 "0ATO010.V" H 9900 800 60  0001 C CNN "Mfg PN"
-	1    9900 800
-	1    0    0    -1
-$EndComp
-$Comp
-L F_Small F3
+P 10000 800
+F 0 "F1" H 9960 860 50  0000 L CNN
+F 1 "10A" H 9880 740 50  0000 L CNN
+F 2 "IPC_MFG:MPD_BK-6010" H 10000 800 50  0001 C CNN
+F 3 "" H 10000 800 50  0000 C CNN
+F 4 "0ATO010.V" H 10000 800 60  0001 C CNN "Mfg PN"
+	1    10000 800
+	1    0    0    -1
+$EndComp
+$Comp
+L FUSE F3
 U 1 1 57D11A86
-P 9900 1900
-F 0 "F3" H 9860 1960 50  0000 L CNN
-F 1 "5A" H 9780 1840 50  0000 L CNN
-F 2 "IPC_MFG:MPD_BK-6010" H 9900 1900 50  0001 C CNN
-F 3 "" H 9900 1900 50  0000 C CNN
-F 4 "0ATO005.V" H 9900 1900 60  0001 C CNN "Mfg PN"
-	1    9900 1900
-	1    0    0    -1
-$EndComp
-$Comp
-L +12V #PWR045
+P 10000 1900
+F 0 "F3" H 9960 1960 50  0000 L CNN
+F 1 "5A" H 9880 1840 50  0000 L CNN
+F 2 "IPC_MFG:MPD_BK-6010" H 10000 1900 50  0001 C CNN
+F 3 "" H 10000 1900 50  0000 C CNN
+F 4 "0ATO005.V" H 10000 1900 60  0001 C CNN "Mfg PN"
+	1    10000 1900
+	1    0    0    -1
+$EndComp
+$Comp
+L +12V #PWR01
 U 1 1 57D11D02
-P 10100 700
-F 0 "#PWR045" H 10100 550 50  0001 C CNN
-F 1 "+12V" H 10100 840 50  0000 C CNN
-F 2 "" H 10100 700 50  0000 C CNN
-F 3 "" H 10100 700 50  0000 C CNN
-	1    10100 700
-	1    0    0    -1
-$EndComp
-$Comp
-L VCC #PWR046
+P 10350 700
+F 0 "#PWR01" H 10350 550 50  0001 C CNN
+F 1 "+12V" H 10350 840 50  0000 C CNN
+F 2 "" H 10350 700 50  0000 C CNN
+F 3 "" H 10350 700 50  0000 C CNN
+	1    10350 700
+	1    0    0    -1
+$EndComp
+$Comp
+L VCC #PWR02
 U 1 1 57D11D56
-P 10100 1800
-F 0 "#PWR046" H 10100 1650 50  0001 C CNN
-F 1 "VCC" H 10100 1950 50  0000 C CNN
-F 2 "" H 10100 1800 50  0000 C CNN
-F 3 "" H 10100 1800 50  0000 C CNN
-	1    10100 1800
-	1    0    0    -1
-$EndComp
-Wire Wire Line
-	10000 1900 10100 1900
-Wire Wire Line
-	10100 1900 10100 1800
-Wire Wire Line
-	10000 800  10100 800
-Wire Wire Line
-	10100 800  10100 700
+P 10350 1800
+F 0 "#PWR02" H 10350 1650 50  0001 C CNN
+F 1 "VCC" H 10350 1950 50  0000 C CNN
+F 2 "" H 10350 1800 50  0000 C CNN
+F 3 "" H 10350 1800 50  0000 C CNN
+	1    10350 1800
+	1    0    0    -1
+$EndComp
+Wire Wire Line
+	10250 1900 10350 1900
+Wire Wire Line
+	10350 1900 10350 1800
+Wire Wire Line
+	10250 800  10350 800
+Wire Wire Line
+	10350 800  10350 700
 $Comp
 L Q_NMOS_GDS Q3
@@
 $EndComp
 $Comp
-L GND #PWR047
+L GND #PWR03
 U 1 1 57D13BB8
 P 4700 6500
-F 0 "#PWR047" H 4700 6250 50  0001 C CNN
+F 0 "#PWR03" H 4700 6250 50  0001 C CNN
 F 1 "GND" H 4700 6350 50  0000 C CNN
 F 2 "" H 4700 6500 50  0000 C CNN
@@
 $EndComp
 Wire Wire Line
-	4800 5800 4700 5800
+	4700 5800 4800 5800
 Connection ~ 4700 6400
 Wire Wire Line
@@
 Connection ~ 4700 5800
 Wire Wire Line
-	4800 5000 4700 5000
+	4700 5000 4800 5000
 Connection ~ 4700 5000
 Wire Wire Line
@@
 	4500 5600 4500 5900
 Wire Wire Line
-	4800 5400 3900 5400
+	3900 5400 4800 5400
 Wire Wire Line
 	4200 5900 4200 5400
@@
 Connection ~ 3300 4400
 Wire Wire Line
-	4800 4300 3000 4300
+	3000 4300 4800 4300
 Connection ~ 3000 4400
 Wire Wire Line
@@
 Connection ~ 1800 4200
 Wire Wire Line
-	2100 5900 2100 4200
+	2100 4200 2100 5900
 Connection ~ 2100 4200
 Connection ~ 3900 4200
@@
 Connection ~ 6500 4400
 Wire Wire Line
-	6700 3800 6700 3700
+	6700 3700 6700 3800
 Connection ~ 6700 3700
 Wire Wire Line
@@
 	7100 5900 7100 5800
 Wire Wire Line
-	8500 4800 9800 4800
-Wire Wire Line
-	9000 4900 9000 4800
+	9000 4800 9000 4900
 Connection ~ 9000 4800
 Wire Wire Line
-	9300 4900 9300 4800
+	9300 4800 9300 4900
 Connection ~ 9300 4800
 Wire Wire Line
-	9600 4900 9600 4800
+	9600 4800 9600 4900
 Connection ~ 9600 4800
 Connection ~ 1800 6400
@@
 Connection ~ 4500 6400
 Wire Wire Line
-	3900 4500 3900 4200
+	3900 4200 3900 4500
 Wire Wire Line
 	3900 4800 3900 5900
@@
 	7000 4200 7000 4100
 Wire Wire Line
-	7000 3800 7000 3700
+	7000 3700 7000 3800
 Connection ~ 7000 3700
 Wire Wire Line
@@
 	8550 5400 8700 5400
 Wire Wire Line
-	8550 5700 8700 5700
-Wire Wire Line
-	8700 5700 8700 4800
+	8700 5700 8550 5700
+Wire Wire Line
+	8700 4800 8700 5700
 Connection ~ 9300 6400
 Connection ~ 9000 6400
@@
 Connection ~ 6800 6300
 Wire Wire Line
-	7450 6200 7450 6400
+	7450 6400 7450 6200
 Wire Wire Line
 	7100 6300 7100 6200
@@
 	9300 6400 9300 5200
 $Comp
-L F_Small F2
+L FUSE F2
 U 1 1 57D13CDB
-P 9900 4800
-F 0 "F2" H 9860 4860 50  0000 L CNN
-F 1 "5A" H 9780 4740 50  0000 L CNN
-F 2 "IPC_MFG:MPD_BK-6010" H 9900 4800 50  0001 C CNN
-F 3 "" H 9900 4800 50  0000 C CNN
-F 4 "0ATO005.V" H 9900 4800 60  0001 C CNN "Mfg PN"
-	1    9900 4800
-	1    0    0    -1
-$EndComp
-Wire Wire Line
-	10000 4800 10100 4800
-Wire Wire Line
-	10100 4800 10100 4700
+P 10000 4800
+F 0 "F2" H 9960 4860 50  0000 L CNN
+F 1 "5A" H 9880 4740 50  0000 L CNN
+F 2 "IPC_MFG:MPD_BK-6010" H 10000 4800 50  0001 C CNN
+F 3 "" H 10000 4800 50  0000 C CNN
+F 4 "0ATO005.V" H 10000 4800 60  0001 C CNN "Mfg PN"
+	1    10000 4800
+	1    0    0    -1
+$EndComp
+Wire Wire Line
+	10250 4800 10350 4800
+Wire Wire Line
+	10350 4800 10350 4700
 Wire Wire Line
 	1500 1300 4800 1300
@@
 	1200 800  1200 3700
 $Comp
-L +5V #PWR048
+L +5V #PWR04
 U 1 1 57D17BA3
 P 3900 700
-F 0 "#PWR048" H 3900 550 50  0001 C CNN
+F 0 "#PWR04" H 3900 550 50  0001 C CNN
 F 1 "+5V" H 3900 840 50  0000 C CNN
 F 2 "" H 3900 700 50  0000 C CNN
@@
 	3900 1600 3900 700
 $Comp
-L +5V #PWR049
+L +5V #PWR05
 U 1 1 57D17EAF
-P 10100 4700
-F 0 "#PWR049" H 10100 4550 50  0001 C CNN
-F 1 "+5V" H 10100 4840 50  0000 C CNN
-F 2 "" H 10100 4700 50  0000 C CNN
-F 3 "" H 10100 4700 50  0000 C CNN
-	1    10100 4700
+P 10350 4700
+F 0 "#PWR05" H 10350 4550 50  0001 C CNN
+F 1 "+5V" H 10350 4840 50  0000 C CNN
+F 2 "" H 10350 4700 50  0000 C CNN
+F 3 "" H 10350 4700 50  0000 C CNN
+	1    10350 4700
 	1    0    0    -1
 $EndComp
@@
 PGD3
 $Comp
-L +12V #PWR050
+L +12V #PWR06
 U 1 1 57D62CC6
 P 2200 6900
-F 0 "#PWR050" H 2200 6750 50  0001 C CNN
+F 0 "#PWR06" H 2200 6750 50  0001 C CNN
 F 1 "+12V" H 2200 7040 50  0000 C CNN
 F 2 "" H 2200 6900 50  0000 C CNN
@@
 PGD3
 $Comp
-L GND #PWR051
+L GND #PWR07
 U 1 1 57D64C7F
 P 1200 7700
-F 0 "#PWR051" H 1200 7450 50  0001 C CNN
+F 0 "#PWR07" H 1200 7450 50  0001 C CNN
 F 1 "GND" H 1200 7550 50  0000 C CNN
 F 2 "" H 1200 7700 50  0000 C CNN
@@
 Wire Wire Line
 	2200 6900 2200 7600
+Text Label 1600 800  0    50   ~ 0
+12VIN
+Wire Wire Line
+	8500 1900 9750 1900
+Wire Wire Line
+	8500 4800 9750 4800
+Text Label 9000 4800 0    50   ~ 0
+5VOUT
+Text Label 9000 1900 0    50   ~ 0
+3V3OUT
 $EndSCHEMATC

Commit message: Update 1/1/2017
Parts:
- R2: value 2k5 -> 1k
Changed lines of the file:
@@
 P 3900 3150
 F 0 "R2" V 3980 3150 50  0000 C CNN
-F 1 "2k5" V 3900 3150 50  0000 C CNN
+F 1 "1k" V 3900 3150 50  0000 C CNN
 F 2 "IPC_RES:RESC1608X55N" V 3830 3150 50  0001 C CNN
 F 3 "" H 3900 3150 50  0000 C CNN

Commit message: Changed Power management
Parts:
- removed C1, C2, C23, C3, C4, C5: 10u, IPC_CAP:CAPC1608X95N, symbol C
- removed C10, C11, C7: 0u1, IPC_CAP:CAPC1608X90N, symbol C
- removed C12: 180n, IPC_CAP:CAPC1608X90N, symbol C
- removed C13: 62p, IPC_CAP:CAPC1608X90N, symbol C
- removed C14: 1n3, IPC_CAP:CAPC1608X90N, symbol C
- removed C15: 5n6, IPC_CAP:CAPC1608X90N, symbol C
- removed C16, C17, C18: 150u, IPC_CAP:CAPAE660X770N, symbol CP1
- removed C6: 4u7, IPC_CAP:CAPC1608X95N, symbol C
- removed C8: 2u2, IPC_CAP:CAPC1608X90N, symbol C
- removed C9: 10n, IPC_CAP:CAPC1608X90N, symbol C
- removed D1: PMEG3050EP,115, IPC_SOD:SOD4725X100N, symbol D_Schottky
- removed F3: 5A, IPC_MFG:MPD_BK-6010, symbol FUSE
- removed L1: 6u8, IPC_IND:INDM1213X620N, symbol INDUCTOR
- removed Q1, Q2, Q3, Q4: STD86N3LH5, IPC_TO:TO228P972X240-3N, symbol Q_NMOS_GDS
- removed R1, R6: 10k, IPC_RES:RESC1608X55N, symbol R
- removed R2: 1k, IPC_RES:RESC1608X55N, symbol R
- removed R3: 499R, IPC_RES:RESC1608X55N, symbol R
- removed R4: 56k2, IPC_RES:RESC1608X55N, symbol R
- removed R5: 2k21, IPC_RES:RESC1608X55N, symbol R
- removed R7: 196R, IPC_RES:RESC1608X55N, symbol R
- removed U1, U2: ISL6420B, IPC_SOP:SOP63P600X155-20N, symbol ISL6420B
- added C19, C20: 1u, IPC_CAP:CAPC1608X90N, symbol C
- added Q1, Q2: SI7386DP, IPC_SON:SON9P127_490X590X112L61X41T376X348N, symbol Q_NMOS_DDDDGSSSD
- added Q3, Q4: RE1J002YNTCL, IPC_SOFL:SOTFL3P50_160X85L45X28N, symbol Q_NMOS_GSD
- added R8, R9: 10k, IPC_RES:RESC1608X55N, symbol R
- added U1: ISL6420BIRZ, IPC_QFN:QFN21P50_400X400X100L55X24T210N, symbol ISL6420BIRZ
- added U2: LP38693SD, IPC_SON:SON7P95_300X300X80L40X35T210X160N, symbol LP38693SD
- C14: renamed from C32; value 1n5 -> 1n3
- C15: renamed from C33; value 6n2 -> 5n6
- L1: renamed from L2; value 8u2 -> 6u8
- R3: renamed from R10; value 510R -> 665R
- R6: renamed from R14; value 178R -> 191R
- renumbered C19 to C1, C28 to C10, C29 to C11, C30 to C12, C31 to C13, C34 to C16, C35 to C17, C36 to C18, C20 to C2, C21 to C3, C22 to C4, C24 to C6, C25 to C7, C26 to C8, C27 to C9, D2 to D1, D3 to D2, D4 to D3, D5 to D4, R8 to R1, R34 to R10, R35 to R11, R36 to R12, R9 to R2, R13 to R4, R12 to R5, R11 to R7
Connections:
- net labels added: BOOT, COMP, DLY, EN, FB, LG, OVP, PG5, PH, REF, UG, VCC5, Z1, Z2
- net labels removed: 3V3OUT
- wire segments 194 -> 136
Other:
- moved on the sheet: C1, C10, C11, C12, C13, C14, C15, C16, C17, C18, C2, C3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

Commit message: KiCAD 4.0.5 Update corrections
Other:
- moved on the sheet: D2, D3, D4
Changed lines of the file:
@@
 LIBS:microcontrollers
 LIBS:dsp
-LIBS:microchip
+LIBS:Microchip Technologies
 LIBS:analog_switches
 LIBS:motorola
-LIBS:texas
+LIBS:TI
 LIBS:intel
 LIBS:audio
@@
 LIBS:stepstick
 LIBS:Linear Technologies
-LIBS:Microchip Technologies
 LIBS:Maxim Integrated
 LIBS:Intersil
 LIBS:mounting hole
-LIBS:TI
 LIBS:power_transistors
 LIBS:FireMC-3.14-cache
@@
 L LED D2
 U 1 1 57D606BA
-P 2800 6200
-F 0 "D2" H 2800 6300 50  0000 C CNN
-F 1 "LED" H 2800 6100 50  0000 C CNN
-F 2 "IPC_LED:LEDM1608X70N" H 2800 6200 50  0001 C CNN
-F 3 "" H 2800 6200 50  0000 C CNN
-	1    2800 6200
+P 2750 6200
+AR Path="/57D606BA" Ref="D2"  Part="1"
+AR Path="/57C8E291/57D606BA" Ref="D2"  Part="1"
+F 0 "D2" H 2750 6300 50  0000 C CNN
+F 1 "LED" H 2750 6100 50  0000 C CNN
+F 2 "IPC_LED:LEDM1608X70N" H 2750 6200 50  0001 C CNN
+F 3 "" H 2750 6200 50  0000 C CNN
+	1    2750 6200
 	1    0    0    1
 $EndComp
@@
 L LED D3
 U 1 1 57D607A1
-P 2800 6500
-F 0 "D3" H 2800 6600 50  0000 C CNN
-F 1 "LED" H 2800 6400 50  0000 C CNN
-F 2 "IPC_LED:LEDM1608X70N" H 2800 6500 50  0001 C CNN
-F 3 "" H 2800 6500 50  0000 C CNN
-	1    2800 6500
+P 2750 6500
+AR Path="/57D607A1" Ref="D3"  Part="1"
+AR Path="/57C8E291/57D607A1" Ref="D3"  Part="1"
+F 0 "D3" H 2750 6600 50  0000 C CNN
+F 1 "LED" H 2750 6400 50  0000 C CNN
+F 2 "IPC_LED:LEDM1608X70N" H 2750 6500 50  0001 C CNN
+F 3 "" H 2750 6500 50  0000 C CNN
+	1    2750 6500
 	1    0    0    1
 $EndComp
@@
 L LED D4
 U 1 1 57D60886
-P 2800 6800
-F 0 "D4" H 2800 6900 50  0000 C CNN
-F 1 "LED" H 2800 6700 50  0000 C CNN
-F 2 "IPC_LED:LEDM1608X70N" H 2800 6800 50  0001 C CNN
-F 3 "" H 2800 6800 50  0000 C CNN
-	1    2800 6800
+P 2750 6800
+AR Path="/57D60886" Ref="D4"  Part="1"
+AR Path="/57C8E291/57D60886" Ref="D4"  Part="1"
+F 0 "D4" H 2750 6900 50  0000 C CNN
+F 1 "LED" H 2750 6700 50  0000 C CNN
+F 2 "IPC_LED:LEDM1608X70N" H 2750 6800 50  0001 C CNN
+F 3 "" H 2750 6800 50  0000 C CNN
+	1    2750 6800
 	1    0    0    1
 $EndComp
@@
 	2500 6200 2600 6200
 Wire Wire Line
-	3100 6500 3000 6500
-Connection ~ 3100 6200
-Wire Wire Line
-	3100 6800 3000 6800
-Connection ~ 3100 6500
+	3000 6500 2900 6500
+Connection ~ 3000 6200
+Wire Wire Line
+	3000 6800 2900 6800
+Connection ~ 3000 6500
 Wire Wire Line
 	4700 2300 1000 2300
 Wire Wire Line
-	3100 6000 3100 6800
+	3000 6000 3000 6800
 Text Label 1600 900  0    50   ~ 0
 12VIN
@@
 L +12V #PWR05
 U 1 1 58960B20
-P 3100 6000
-F 0 "#PWR05" H 3100 5850 50  0001 C CNN
-F 1 "+12V" H 3100 6140 50  0000 C CNN
-F 2 "" H 3100 6000 50  0000 C CNN
-F 3 "" H 3100 6000 50  0000 C CNN
-	1    3100 6000
+P 3000 6000
+F 0 "#PWR05" H 3000 5850 50  0001 C CNN
+F 1 "+12V" H 3000 6140 50  0000 C CNN
+F 2 "" H 3000 6000 50  0000 C CNN
+F 3 "" H 3000 6000 50  0000 C CNN
+	1    3000 6000
 	1    0    0    -1
 $EndComp
@@
 	2100 7700 2100 6200
 Wire Wire Line
-	3000 6200 3100 6200
+	2900 6200 3000 6200
 Wire Wire Line
 	1200 4300 1500 4300
