File: FireMC-3.14_PWR.sch (KiCad schematic (older format))
At the start: 46 parts, among them J1 Header_1X2, J2 Header_1X2, Q1 SI7386DP, Q2 SI7386DP, Q3 RE1J002YNTCL, Q4 RE1J002YNTCL, U1 ISL6420BIRZ, U2 LP38693SD

Commit message: update
Parts:
- removed U1: ISL6420BIRZ, IPC_QFN:QFN21P50_400X400X100L55X24T210N, symbol ISL6420BIRZ
- added U1: ISL6420BIAZ, IPC_SOP:SOP63P600X155-20N, symbol ISL6420BIAZ
Connections:
- net 12VIN: now also U1.14 (VIN)
- net BOOT: now also U1.7 (BOOT)
- net COMP: now also U1.18 (COMP)
- net DLY: now also U1.1 (CDEL)
- net EN: now also U1.19 (ENSS)
- net FB: now also U1.17 (FB)
- net GND: now also U1.12 (VMSET/MODE), U1.15 (SGND), U1.2 (PGND), U1.8 (GPIO2), U1.9 (GPIO1/REFIN)
- net LG: now also U1.3 (LGATE)
- net OVP: now also U1.10 (OCSET)
- net PG5: now also U1.20 (PGOOD)
- net PH: now also U1.5 (PHASE)
- net REF: now also U1.11 (REFOUT)
- net UG: now also U1.6 (UGATE)
- net VCC5: now also U1.13 (VCC5), U1.16 (RT), U1.4 (PVCC)
Changed lines of the file:
@@
 	10150 900  10250 900
 Wire Wire Line
-	10250 900  10250 800
+	10250 800  10250 1000
 $Comp
 L C C7
@@
 	10150 2000 10250 2000
 Wire Wire Line
-	10250 2000 10250 1900
+	10250 1900 10250 2100
 $Comp
 L Q_NMOS_DDDDGSSSD Q1
@@
 Wire Wire Line
 	9650 900  1100 900
-$Comp
-L ISL6420BIRZ U1
-U 1 1 589A566B
-P 5500 2200
-F 0 "U1" H 6050 3150 60  0000 R CNN
-F 1 "ISL6420BIRZ" H 6050 1250 60  0000 R CNN
-F 2 "IPC_QFN:QFN21P50_400X400X100L55X24T210N" H 4600 2250 60  0001 C CNN
-F 3 "" H 4600 2250 60  0000 C CNN
-	1    5500 2200
-	1    0    0    -1
-$EndComp
 Text Label 3450 1500 0    50   ~ 0
 VCC5
@@
 Text Label 8200 2900 0    50   ~ 0
 Z2
-Wire Wire Line
-	5300 3300 5300 3600
-Connection ~ 5300 3600
+$Comp
+L ISL6420BIAZ U1
+U 1 1 591E516B
+P 5500 2200
+F 0 "U1" H 6050 3150 60  0000 R CNN
+F 1 "ISL6420BIAZ" H 6050 1250 60  0000 R CNN
+F 2 "IPC_SOP:SOP63P600X155-20N" H 4600 2250 60  0001 C CNN
+F 3 "" H 4600 2250 60  0000 C CNN
+	1    5500 2200
+	1    0    0    -1
+$EndComp
+$Comp
+L PWR_FLAG #FLG015
+U 1 1 591E7F63
+P 10250 1000
+F 0 "#FLG015" H 10250 1075 50  0001 C CNN
+F 1 "PWR_FLAG" H 10250 1150 50  0000 C CNN
+F 2 "" H 10250 1000 50  0001 C CNN
+F 3 "" H 10250 1000 50  0001 C CNN
+	1    10250 1000
+	-1   0    0    1
+$EndComp
+$Comp
+L PWR_FLAG #FLG016
+U 1 1 591E7FD3
+P 10250 2100
+F 0 "#FLG016" H 10250 2175 50  0001 C CNN
+F 1 "PWR_FLAG" H 10250 2250 50  0000 C CNN
+F 2 "" H 10250 2100 50  0001 C CNN
+F 3 "" H 10250 2100 50  0001 C CNN
+	1    10250 2100
+	-1   0    0    1
+$EndComp
+Connection ~ 10250 900
+Connection ~ 10250 2000
 $EndSCHEMATC
