File: FireMC-3.14_SFTY.sch (KiCad schematic (older format))
At the start: 6 parts, among them J5 Header_1X2, U5 74LVC1G14, U6 74LV32

Commit message: Time to Update.  Board layout started.
Parts:
- renumbered U5 to U7, U6 to U8
Changed lines of the file:
@@
 LIBS:Maxim Integrated
 LIBS:Intersil
+LIBS:mounting hole
 LIBS:FireMC-3.14-cache
 EELAYER 25 0
@@
 $EndDescr
 $Comp
-L 74AHC1G14 U5
+L 74AHC1G14 U7
 U 1 1 57E0F89D
 P 2650 1850
-F 0 "U5" H 2795 1965 50  0000 C CNN
+F 0 "U7" H 2795 1965 50  0000 C CNN
 F 1 "74LVC1G14" H 2850 1750 50  0000 C CNN
 F 2 "IPC_SOT:SOT95P280X145-5N" H 2745 1715 50  0001 C CNN
@@
 $EndComp
 $Comp
-L 74LS32 U6
+L 74LS32 U8
 U 1 1 57E0F8DC
 P 4300 1750
-F 0 "U6" H 4300 1800 50  0000 C CNN
+F 0 "U8" H 4300 1800 50  0000 C CNN
 F 1 "74LV32" H 4300 1700 50  0000 C CNN
 F 2 "IPC_SOP:SOP65P640X120-14N" H 4300 1750 50  0001 C CNN
@@
 $EndComp
 $Comp
-L 74LS32 U6
+L 74LS32 U8
 U 2 1 57E0F95B
 P 4300 2250
-F 0 "U6" H 4300 2300 50  0000 C CNN
+F 0 "U8" H 4300 2300 50  0000 C CNN
 F 1 "74LV32" H 4300 2200 50  0000 C CNN
 F 2 "IPC_SOP:SOP65P640X120-14N" H 4300 2250 50  0001 C CNN
@@
 $EndComp
 $Comp
-L 74LS32 U6
+L 74LS32 U8
 U 3 1 57E0F976
 P 4300 2750
-F 0 "U6" H 4300 2800 50  0000 C CNN
+F 0 "U8" H 4300 2800 50  0000 C CNN
 F 1 "74LV32" H 4300 2700 50  0000 C CNN
 F 2 "IPC_SOP:SOP65P640X120-14N" H 4300 2750 50  0001 C CNN
@@
 $EndComp
 $Comp
-L 74LS32 U6
+L 74LS32 U8
 U 4 1 57E0F9AB
 P 4300 3250
-F 0 "U6" H 4300 3300 50  0000 C CNN
+F 0 "U8" H 4300 3300 50  0000 C CNN
 F 1 "74LV32" H 4300 3200 50  0000 C CNN
 F 2 "IPC_SOP:SOP65P640X120-14N" H 4300 3250 50  0001 C CNN
@@
 $EndComp
 $Comp
-L GND #PWR052
+L GND #PWR053
 U 1 1 57E11002
 P 1200 2450
-F 0 "#PWR052" H 1200 2200 50  0001 C CNN
+F 0 "#PWR053" H 1200 2200 50  0001 C CNN
 F 1 "GND" H 1200 2300 50  0000 C CNN
 F 2 "" H 1200 2450 50  0000 C CNN
@@
 $EndComp
 $Comp
-L VCC #PWR053
+L VCC #PWR054
 U 1 1 57E11028
 P 2000 1250
-F 0 "#PWR053" H 2000 1100 50  0001 C CNN
+F 0 "#PWR054" H 2000 1100 50  0001 C CNN
 F 1 "VCC" H 2000 1400 50  0000 C CNN
 F 2 "" H 2000 1250 50  0000 C CNN

Commit message: Update 1/1/2017
Parts:
- added MH1, MH2, MH3, MH4, MH5, MH6, MH7, MH8: MountHole_NoElec, IPC_MFG:IMELLC_MH275X600NPTH, symbol MountHole_NoElec
Changed lines of the file:
@@
 $EndComp
 $Comp
-L GND #PWR053
+L GND #PWR052
 U 1 1 57E11002
 P 1200 2450
-F 0 "#PWR053" H 1200 2200 50  0001 C CNN
+F 0 "#PWR052" H 1200 2200 50  0001 C CNN
 F 1 "GND" H 1200 2300 50  0000 C CNN
 F 2 "" H 1200 2450 50  0000 C CNN
@@
 $EndComp
 $Comp
-L VCC #PWR054
+L VCC #PWR053
 U 1 1 57E11028
 P 2000 1250
-F 0 "#PWR054" H 2000 1100 50  0001 C CNN
+F 0 "#PWR053" H 2000 1100 50  0001 C CNN
 F 1 "VCC" H 2000 1400 50  0000 C CNN
 F 2 "" H 2000 1250 50  0000 C CNN
@@
 Wire Notes Line
 	5500 3700 500  3700
+$Comp
+L MountHole_NoElec MH5
+U 1 1 580A60A7
+P 9750 900
+F 0 "MH5" H 9750 1000 50  0000 C CNN
+F 1 "MountHole_NoElec" H 9750 800 50  0000 C CNN
+F 2 "IPC_MFG:IMELLC_MH275X600NPTH" H 9750 900 50  0001 C CNN
+F 3 "" H 9750 900 50  0000 C CNN
+	1    9750 900
+	1    0    0    -1
+$EndComp
+$Comp
+L MountHole_NoElec MH1
+U 1 1 580A6102
+P 9000 900
+F 0 "MH1" H 9000 1000 50  0000 C CNN
+F 1 "MountHole_NoElec" H 9000 800 50  0000 C CNN
+F 2 "IPC_MFG:IMELLC_MH275X600NPTH" H 9000 900 50  0001 C CNN
+F 3 "" H 9000 900 50  0000 C CNN
+	1    9000 900
+	1    0    0    -1
+$EndComp
+$Comp
+L MountHole_NoElec MH2
+U 1 1 580A6153
+P 9000 1200
+F 0 "MH2" H 9000 1300 50  0000 C CNN
+F 1 "MountHole_NoElec" H 9000 1100 50  0000 C CNN
+F 2 "IPC_MFG:IMELLC_MH275X600NPTH" H 9000 1200 50  0001 C CNN
+F 3 "" H 9000 1200 50  0000 C CNN
+	1    9000 1200
+	1    0    0    -1
+$EndComp
+$Comp
+L MountHole_NoElec MH6
+U 1 1 580A618F
+P 9750 1200
+F 0 "MH6" H 9750 1300 50  0000 C CNN
+F 1 "MountHole_NoElec" H 9750 1100 50  0000 C CNN
+F 2 "IPC_MFG:IMELLC_MH275X600NPTH" H 9750 1200 50  0001 C CNN
+F 3 "" H 9750 1200 50  0000 C CNN
+	1    9750 1200
+	1    0    0    -1
+$EndComp
+$Comp
+L MountHole_NoElec MH7
+U 1 1 580A61D8
+P 9750 1500
+F 0 "MH7" H 9750 1600 50  0000 C CNN
+F 1 "MountHole_NoElec" H 9750 1400 50  0000 C CNN
+F 2 "IPC_MFG:IMELLC_MH275X600NPTH" H 9750 1500 50  0001 C CNN
+F 3 "" H 9750 1500 50  0000 C CNN
+	1    9750 1500
+	1    0    0    -1
+$EndComp
+$Comp
+L MountHole_NoElec MH3
+U 1 1 580A621A
+P 9000 1500
+F 0 "MH3" H 9000 1600 50  0000 C CNN
+F 1 "MountHole_NoElec" H 9000 1400 50  0000 C CNN
+F 2 "IPC_MFG:IMELLC_MH275X600NPTH" H 9000 1500 50  0001 C CNN
+F 3 "" H 9000 1500 50  0000 C CNN
+	1    9000 1500
+	1    0    0    -1
+$EndComp
+$Comp
+L MountHole_NoElec MH4
+U 1 1 580A627F
+P 9000 1800
+F 0 "MH4" H 9000 1900 50  0000 C CNN
+F 1 "MountHole_NoElec" H 9000 1700 50  0000 C CNN
+F 2 "IPC_MFG:IMELLC_MH275X600NPTH" H 9000 1800 50  0001 C CNN
+F 3 "" H 9000 1800 50  0000 C CNN
+	1    9000 1800
+	1    0    0    -1
+$EndComp
+$Comp
+L MountHole_NoElec MH8
+U 1 1 580A62CB
+P 9750 1800
+F 0 "MH8" H 9750 1900 50  0000 C CNN
+F 1 "MountHole_NoElec" H 9750 1700 50  0000 C CNN
+F 2 "IPC_MFG:IMELLC_MH275X600NPTH" H 9750 1800 50  0001 C CNN
+F 3 "" H 9750 1800 50  0000 C CNN
+	1    9750 1800
+	1    0    0    -1
+$EndComp
 $EndSCHEMATC

Commit message: Changed Power management
Parts:
- renumbered C39 to C25, J5 to J20, MH5 to MH2, MH2 to MH3, MH6 to MH4, MH3 to MH5, MH7 to MH6, MH4 to MH7, R16 to R30, R15 to R31, U7 to U9
Changed lines of the file:
@@
 LIBS:Intersil
 LIBS:mounting hole
+LIBS:TI
+LIBS:power_transistors
 LIBS:FireMC-3.14-cache
 EELAYER 25 0
@@
 $EndDescr
 $Comp
-L 74AHC1G14 U7
+L 74AHC1G14 U9
 U 1 1 57E0F89D
 P 2650 1850
-F 0 "U7" H 2795 1965 50  0000 C CNN
+F 0 "U9" H 2795 1965 50  0000 C CNN
 F 1 "74LVC1G14" H 2850 1750 50  0000 C CNN
 F 2 "IPC_SOT:SOT95P280X145-5N" H 2745 1715 50  0001 C CNN
@@
 $EndComp
 $Comp
-L C C39
+L C C25
 U 1 1 57E0F9CE
 P 2000 2100
-F 0 "C39" H 2025 2200 50  0000 L CNN
+F 0 "C25" H 2025 2200 50  0000 L CNN
 F 1 "2u2" H 2025 2000 50  0000 L CNN
 F 2 "IPC_CAP:CAPC1608X90N" H 2038 1950 50  0001 C CNN
@@
 $EndComp
 $Comp
-L R R16
+L R R30
 U 1 1 57E0FA43
 P 2000 1600
-F 0 "R16" V 2080 1600 50  0000 C CNN
+F 0 "R30" V 2080 1600 50  0000 C CNN
 F 1 "3k3" V 2000 1600 50  0000 C CNN
 F 2 "IPC_RES:RESC1608X55N" V 1930 1600 50  0001 C CNN
@@
 $EndComp
 $Comp
-L R R15
+L R R31
 U 1 1 57E0FAB4
 P 1450 1850
-F 0 "R15" V 1530 1850 50  0000 C CNN
+F 0 "R31" V 1530 1850 50  0000 C CNN
 F 1 "330R" V 1450 1850 50  0000 C CNN
 F 2 "IPC_RES:RESC1608X55N" V 1380 1850 50  0001 C CNN
@@
 $EndComp
 $Comp
-L Header_1X2 J5
+L Header_1X2 J20
 U 1 1 57E0FAEF
 P 800 1900
-F 0 "J5" H 800 2100 60  0000 C CNN
+F 0 "J20" H 800 2100 60  0000 C CNN
 F 1 "Header_1X2" H 800 1700 60  0000 C CNN
 F 2 "IPC_MFG:SULLINS_PRPC002SAAN-RC" H 800 1800 60  0001 C CNN
@@
 $EndComp
 $Comp
-L GND #PWR052
+L GND #PWR059
 U 1 1 57E11002
 P 1200 2450
-F 0 "#PWR052" H 1200 2200 50  0001 C CNN
+F 0 "#PWR059" H 1200 2200 50  0001 C CNN
 F 1 "GND" H 1200 2300 50  0000 C CNN
 F 2 "" H 1200 2450 50  0000 C CNN
@@
 $EndComp
 $Comp
-L VCC #PWR053
+L VCC #PWR060
 U 1 1 57E11028
 P 2000 1250
-F 0 "#PWR053" H 2000 1100 50  0001 C CNN
+F 0 "#PWR060" H 2000 1100 50  0001 C CNN
 F 1 "VCC" H 2000 1400 50  0000 C CNN
 F 2 "" H 2000 1250 50  0000 C CNN
@@
 	5500 3700 500  3700
 $Comp
-L MountHole_NoElec MH5
+L MountHole_NoElec MH2
 U 1 1 580A60A7
 P 9750 900
-F 0 "MH5" H 9750 1000 50  0000 C CNN
+F 0 "MH2" H 9750 1000 50  0000 C CNN
 F 1 "MountHole_NoElec" H 9750 800 50  0000 C CNN
 F 2 "IPC_MFG:IMELLC_MH275X600NPTH" H 9750 900 50  0001 C CNN
@@
 $EndComp
 $Comp
-L MountHole_NoElec MH2
+L MountHole_NoElec MH3
 U 1 1 580A6153
 P 9000 1200
-F 0 "MH2" H 9000 1300 50  0000 C CNN
+F 0 "MH3" H 9000 1300 50  0000 C CNN
 F 1 "MountHole_NoElec" H 9000 1100 50  0000 C CNN
 F 2 "IPC_MFG:IMELLC_MH275X600NPTH" H 9000 1200 50  0001 C CNN
@@
 $EndComp
 $Comp
-L MountHole_NoElec MH6
+L MountHole_NoElec MH4
 U 1 1 580A618F
 P 9750 1200
-F 0 "MH6" H 9750 1300 50  0000 C CNN
+F 0 "MH4" H 9750 1300 50  0000 C CNN
 F 1 "MountHole_NoElec" H 9750 1100 50  0000 C CNN
 F 2 "IPC_MFG:IMELLC_MH275X600NPTH" H 9750 1200 50  0001 C CNN
@@
 $EndComp
 $Comp
-L MountHole_NoElec MH7
+L MountHole_NoElec MH6
 U 1 1 580A61D8
 P 9750 1500
-F 0 "MH7" H 9750 1600 50  0000 C CNN
+F 0 "MH6" H 9750 1600 50  0000 C CNN
 F 1 "MountHole_NoElec" H 9750 1400 50  0000 C CNN
 F 2 "IPC_MFG:IMELLC_MH275X600NPTH" H 9750 1500 50  0001 C CNN
@@
 $EndComp
 $Comp
-L MountHole_NoElec MH3
+L MountHole_NoElec MH5
 U 1 1 580A621A
 P 9000 1500
-F 0 "MH3" H 9000 1600 50  0000 C CNN
+F 0 "MH5" H 9000 1600 50  0000 C CNN
 F 1 "MountHole_NoElec" H 9000 1400 50  0000 C CNN
 F 2 "IPC_MFG:IMELLC_MH275X600NPTH" H 9000 1500 50  0001 C CNN
@@
 $EndComp
 $Comp
-L MountHole_NoElec MH4
+L MountHole_NoElec MH7
 U 1 1 580A627F
 P 9000 1800
-F 0 "MH4" H 9000 1900 50  0000 C CNN
+F 0 "MH7" H 9000 1900 50  0000 C CNN
 F 1 "MountHole_NoElec" H 9000 1700 50  0000 C CNN
 F 2 "IPC_MFG:IMELLC_MH275X600NPTH" H 9000 1800 50  0001 C CNN
